Commit message: 0326

File: urdf/depth_camera.xacro (robot description, xacro)
@@ -20,5 +20,5 @@
             </camera>
             <plugin name="camera_controller" filename="libgazebo_ros_camera.so">
-                <frame_name>camera_link_optical</frame_name>
+                <frame_name>camera_optical_link</frame_name>
                 <min_depth>0.1</min_depth>
                 <max_depth>100.0</max_depth>

File: urdf/robot_core.xacro (robot description, xacro)
@@ -32,5 +32,5 @@
     <xacro:property name="caster_wheel_mass" value="0.5"/>
     <!-- Update All Parameters from a Single Parameter -->
-    <xacro:property name="scale" value="10.0"/>
+    <xacro:property name="scale" value="20.0"/>
     <xacro:property name="scaled_chassis_radius" value="${chassis_radius * scale}"/>
     <xacro:property name="scaled_chassis_length" value="${chassis_length * scale}"/>
@@ -171,7 +171,7 @@
     <joint name="camera_optical_joint" type="fixed">
         <parent link="camera_link"/>
-        <child link="camera_link_optical"/>
+        <child link="camera_optical_link"/>
         <origin xyz="0 0 0" rpy="${-pi/2} 0 ${-pi/2}"/>
     </joint>
-    <link name="camera_link_optical"/>
+    <link name="camera_optical_link"/>
 </robot>
