Commit message: 0326

File: urdf/robot_core.xacro (robot description, xacro)
@@ -135,5 +135,5 @@
         <visual>
             <geometry>
-                <sphere radius="${scaled_wheel_radius / 1.5}"/>
+                <sphere radius="${scaled_wheel_radius / 2}"/>
             </geometry>
             <material name="black"/>
@@ -141,8 +141,8 @@
         <collision>
             <geometry>
-                <sphere radius="${scaled_wheel_radius / 1.5}"/>
+                <sphere radius="${scaled_wheel_radius / 2}"/>
             </geometry>
         </collision>
-        <xacro:inertial_sphere mass="${scaled_caster_wheel_mass}" radius="${scaled_wheel_radius / 1.5}">
+        <xacro:inertial_sphere mass="${scaled_caster_wheel_mass}" radius="${scaled_wheel_radius / 2}">
             <origin xyz="0 0 0" rpy="0 0 0"/>
         </xacro:inertial_sphere>
