Commit message: 0326

File: urdf/gazebo_control.xacro (robot description, xacro)
@@ -6,4 +6,6 @@
             <left_joint>left_wheel_joint</left_joint>
             <right_joint>right_wheel_joint</right_joint>
+            <!-- <wheel_separation>${2 * scaled_chassis_radius + scaled_wheel_length}</wheel_separation>
+            <wheel_diameter>${scaled_wheel_radius}</wheel_diameter> -->
             <wheel_separation>0.35</wheel_separation>
             <wheel_diameter>0.1</wheel_diameter>

File: urdf/rgb_camera.xacro (robot description, xacro)
@@ -3,5 +3,5 @@
     <gazebo reference="camera_link">
         <material>Gazebo/Red</material>
-        <sensor name="camera" type="depth">
+        <sensor name="camera" type="camera">
             <pose>0 0 0 0 0 0</pose>
             <visualize>true</visualize>
@@ -20,4 +20,5 @@
             </camera>
             <plugin name="camera_controller" filename="libgazebo_ros_camera.so">
+                <alwaysOn>true</alwaysOn>
                 <frame_name>camera_optical_link</frame_name>
                 <min_depth>0.1</min_depth>

File: urdf/robot_core.xacro (robot description, xacro)
@@ -4,5 +4,7 @@
     <xacro:include filename="inertial_macros.xacro"/>
     <!-- CAMERA PARAMETERS -->
-    <xacro:include filename="depth_camera.xacro"/>
+    <!-- <xacro:include filename="depth_camera.xacro"/> -->
+    <xacro:include filename="rgb_camera.xacro"/>
+    <!-- <xacro:include filename="gazebo_control.xacro"/> -->
     <!-- COLORS -->
     <material name="white">
@@ -24,17 +26,20 @@
     <link name="base_link"/>
     <!-- DEFINE PARAMETERS -->
-    <xacro:property name="chassis_radius" value="0.02"/>
-    <xacro:property name="chassis_length" value="0.1"/>
-    <xacro:property name="wheel_radius" value="0.025"/>
-    <xacro:property name="wheel_length" value="0.01"/>
-    <xacro:property name="chassis_mass" value="0.5"/>
-    <xacro:property name="wheel_mass" value="0.1"/>
-    <xacro:property name="caster_wheel_mass" value="0.5"/>
+    <xacro:property name="chassis_radius" value="0.0065"/>
+    <xacro:property name="chassis_length" value="0.02"/>
+    <xacro:property name="wheel_radius" value="0.008"/>
+    <xacro:property name="wheel_length" value="0.001"/>
+    <xacro:property name="chassis_mass" value="0.002"/>
+    <xacro:property name="wheel_mass" value="0.001"/>
+    <xacro:property name="caster_wheel_mass" value="0.01"/>
     <!-- Update All Parameters from a Single Parameter -->
-    <xacro:property name="scale" value="20.0"/>
+    <xacro:property name="scale" value="50.0"/>
     <xacro:property name="scaled_chassis_radius" value="${chassis_radius * scale}"/>
     <xacro:property name="scaled_chassis_length" value="${chassis_length * scale}"/>
-    <xacro:property name="scaled_wheel_radius" value="${wheel_radius * scale}"/>
+    <xacro:property name="scaled_wheel_radius" value="${scaled_chassis_radius * 1.1}"/>
     <xacro:property name="scaled_wheel_length" value="${wheel_length * scale}"/>
+    <xacro:property name="scaled_chassis_mass" value="${chassis_mass * scale}"/>
+    <xacro:property name="scaled_wheel_mass" value="${wheel_mass * scale}"/>
+    <xacro:property name="scaled_caster_wheel_mass" value="${caster_wheel_mass * scale}"/>
     <xacro:property name="scaled_camera_length" value="${scaled_chassis_radius / 5}"/>
     <!-- CHASSIS LINK -->
@@ -58,5 +63,5 @@
             </geometry>
         </collision>
-        <xacro:inertial_cylinder mass="${chassis_mass}" radius="${scaled_chassis_radius}" length="${scaled_chassis_length}">
+        <xacro:inertial_cylinder mass="${scaled_chassis_mass}" radius="${scaled_chassis_radius}" length="${scaled_chassis_length}">
             <origin xyz="0 0 0" rpy="0 ${pi/2} 0"/>
         </xacro:inertial_cylinder>
@@ -86,5 +91,5 @@
             </geometry>
         </collision>
-        <xacro:inertial_cylinder mass="${wheel_mass}" radius="${scaled_wheel_radius}" length="${scaled_wheel_length}">
+        <xacro:inertial_cylinder mass="${scaled_wheel_mass}" radius="${scaled_wheel_radius}" length="${scaled_wheel_length}">
             <origin xyz="0 0 ${scaled_wheel_length / 2}" rpy="0 0 0"/>
         </xacro:inertial_cylinder>
@@ -114,5 +119,5 @@
             </geometry>
         </collision>
-        <xacro:inertial_cylinder mass="${wheel_mass}" radius="${scaled_wheel_radius}" length="${scaled_wheel_length}">
+        <xacro:inertial_cylinder mass="${scaled_wheel_mass}" radius="${scaled_wheel_radius}" length="${scaled_wheel_length}">
             <origin xyz="0 0 ${scaled_wheel_length / 2}" rpy="0 0 0"/>
         </xacro:inertial_cylinder>
@@ -139,5 +144,5 @@
             </geometry>
         </collision>
-        <xacro:inertial_sphere mass="${caster_wheel_mass}" radius="${scaled_wheel_radius / 1.5}">
+        <xacro:inertial_sphere mass="${scaled_caster_wheel_mass}" radius="${scaled_wheel_radius / 1.5}">
             <origin xyz="0 0 0" rpy="0 0 0"/>
         </xacro:inertial_sphere>

Commit message: 0327

File: urdf/gazebo_control.xacro (robot description, xacro)
@@ -4,14 +4,15 @@
         <plugin name="diff_drive" filename="libgazebo_ros_diff_drive.so">
             <!-- Wheel Information -->
-            <left_joint>left_wheel_joint</left_joint>
-            <right_joint>right_wheel_joint</right_joint>
-            <!-- <wheel_separation>${2 * scaled_chassis_radius + scaled_wheel_length}</wheel_separation>
-            <wheel_diameter>${scaled_wheel_radius}</wheel_diameter> -->
-            <wheel_separation>0.35</wheel_separation>
-            <wheel_diameter>0.1</wheel_diameter>
+            <left_joint>lb_wheel_joint</left_joint>
+            <right_joint>rb_wheel_joint</right_joint>
+            <wheel_separation>${2 * scaled_chassis_radius + scaled_wheel_length}</wheel_separation>
+            <wheel_diameter>${scaled_wheel_radius}</wheel_diameter>
+            <!-- <wheel_separation>0.35</wheel_separation>
+            <wheel_diameter>0.1</wheel_diameter> -->
             <!-- Limits -->
             <max_wheel_torque>200</max_wheel_torque>
             <max_wheel_acceleration>10.0</max_wheel_acceleration>
             <!-- Output -->
+            <command_topic>cmd_vel</command_topic>
             <odometry_frame>odom</odometry_frame>
             <robot_base_frame>base_link</robot_base_frame>

File: urdf/robot_core_copy.xacro (robot description, xacro)
@@ -43,11 +43,11 @@
     <xacro:property name="scaled_caster_wheel_mass" value="${caster_wheel_mass * scale}"/>
     <xacro:property name="scaled_camera_length" value="${scaled_chassis_radius / 5}"/>
-    <!-- BACK CHASSIS LINK -->
-    <joint name="back_chassis_joint" type="fixed">
+    <!-- CHASSIS LINK -->
+    <joint name="chassis_joint" type="fixed">
         <parent link="base_link"/>
-        <child link="back_chassis"/>
+        <child link="chassis"/>
         <origin xyz="${scaled_chassis_length / 2} 0 ${scaled_wheel_radius}" rpy="0 0 0"/>
     </joint>
-    <link name="back_chassis">
+    <link name="chassis">
         <visual>
             <origin xyz="0 0 0" rpy="0 ${pi/2} 0"/>
@@ -60,5 +60,5 @@
             <origin xyz="0 0 0" rpy="0 ${pi/2} 0"/>
             <geometry>
-                <cylinder radius="${scaled_chassis_radius}" length="${scaled_chassis_length * 0.8}"/>
+                <cylinder radius="${scaled_chassis_radius}" length="${scaled_chassis_length}"/>
             </geometry>
         </collision>
@@ -67,15 +67,15 @@
         </xacro:inertial_cylinder>
     </link>
-    <gazebo reference="back_chassis">
+    <gazebo reference="chassis">
         <material>Gazebo/White</material>
     </gazebo>
-    <!-- LEFT BACK WHEEL LINK -->
-    <joint name="lb_wheel_joint" type="continuous">
+    <!-- LEFT WHEEL LINK -->
+    <joint name="left_wheel_joint" type="continuous">
         <parent link="base_link"/>
-        <child link="lb_wheel"/>
+        <child link="left_wheel"/>
         <origin xyz="${scaled_wheel_radius} ${scaled_chassis_radius} ${scaled_wheel_radius}" rpy="-${pi/2} 0 0" />
         <axis xyz="0 0 1"/>
     </joint>
-    <link name="lb_wheel">
+    <link name="left_wheel">
         <visual>
             <origin xyz="0 0 ${scaled_wheel_length / 2}" rpy="0 0 0"/>
@@ -95,15 +95,15 @@
         </xacro:inertial_cylinder>
     </link>
-    <gazebo reference="lb_wheel">
+    <gazebo reference="left_wheel">
         <material>Gazebo/Blue</material>
     </gazebo>
-    <!-- RIGHT BACK WHEEL LINK -->
-    <joint name="rb_wheel_joint" type="continuous">
+    <!-- RIGHT WHEEL LINK -->
+    <joint name="right_wheel_joint" type="continuous">
         <parent link="base_link"/>
-        <child link="rb_wheel"/>
+        <child link="right_wheel"/>
         <origin xyz="${scaled_wheel_radius} -${scaled_chassis_radius} ${scaled_wheel_radius}" rpy="${pi/2} 0 0" />
         <axis xyz="0 0 -1"/>
     </joint>
-    <link name="rb_wheel">
+    <link name="right_wheel">
         <visual>
             <origin xyz="0 0 ${scaled_wheel_length / 2}" rpy="0 0 0"/>
@@ -123,14 +123,14 @@
         </xacro:inertial_cylinder>
     </link>
-    <gazebo reference="rb_wheel">
+    <gazebo reference="right_wheel">
         <material>Gazebo/Blue</material>
     </gazebo>
-    <!-- BACK CASTER WHEEL LINK -->
-    <joint name="b_caster_wheel_joint" type="fixed">
-        <parent link="back_chassis"/>
-        <child link="b_caster_wheel"/>
+    <!-- CASTER WHEEL LINK -->
+    <joint name="caster_wheel_joint" type="fixed">
+        <parent link="chassis"/>
+        <child link="caster_wheel"/>
         <origin xyz="${scaled_chassis_length / 4} 0 -${scaled_wheel_radius / 2}" rpy="0 0 0"/>
     </joint>
-    <link name="b_caster_wheel">
+    <link name="caster_wheel">
         <visual>
             <geometry>
@@ -148,117 +148,5 @@
         </xacro:inertial_sphere>
     </link>
-    <gazebo reference="b_caster_wheel">
-        <material>Gazebo/Black</material>
-        <mu1 value="0.001"/>
-        <mu2 value="0.001"/>
-    </gazebo>
-    <!-- FRONT CHASSIS LINK -->
-    <joint name="joint_between_chassis" type="revolute">
-        <parent link="back_chassis"/>
-        <child link="front_chassis"/>
-        <origin xyz="${scaled_chassis_length} 0 0" rpy="0 0 0"/>
-        <axis xyz="0 1 0"/>
-        <limit velocity="10.0" effort="200" lower="-${pi/2}" upper="${pi/2}"/>
-    </joint>
-    <link name="front_chassis">
-        <visual>
-            <origin xyz="0 0 0" rpy="0 ${pi/2} 0"/>
-            <geometry>
-                <cylinder radius="${scaled_chassis_radius}" length="${scaled_chassis_length}"/>
-            </geometry>
-            <material name="white"/>
-        </visual>
-        <collision>
-            <origin xyz="0 0 0" rpy="0 ${pi/2} 0"/>
-            <geometry>
-                <cylinder radius="${scaled_chassis_radius}" length="${scaled_chassis_length * 0.8}"/>
-            </geometry>
-        </collision>
-        <xacro:inertial_cylinder mass="${scaled_chassis_mass}" radius="${scaled_chassis_radius}" length="${scaled_chassis_length}">
-            <origin xyz="0 0 0" rpy="0 ${pi/2} 0"/>
-        </xacro:inertial_cylinder>
-    </link>
-    <gazebo reference="front_chassis">
-        <material>Gazebo/White</material>
-    </gazebo>
-    <!-- LEFT FRONT WHEEL LINK -->
-    <joint name="lf_wheel_joint" type="continuous">
-        <parent link="front_chassis"/>
-        <child link="lf_wheel"/>
-        <origin xyz="${scaled_wheel_length / 2 - scaled_wheel_radius / 2} ${scaled_chassis_radius} 0" rpy="-${pi/2} 0 0"/>
-        <axis xyz="0 0 1"/>
-    </joint>
-    <link name="lf_wheel">
-        <visual>
-            <origin xyz="0 0 ${scaled_wheel_length / 2}" rpy="0 0 0"/>
-            <geometry>
-                <cylinder radius="${scaled_wheel_radius}" length="${scaled_wheel_length}"/>
-            </geometry>
-            <material name="red"/>
-        </visual>
-        <collision>
-            <origin xyz="0 0 ${scaled_wheel_length / 2}" rpy="0 0 0"/>
-            <geometry>
-                <cylinder radius="${scaled_wheel_radius}" length="${scaled_wheel_length}"/>
-            </geometry>
-        </collision>
-        <xacro:inertial_cylinder mass="${scaled_wheel_mass}" radius="${scaled_wheel_radius}" length="${scaled_wheel_length}">
-            <origin xyz="0 0 ${scaled_wheel_length / 2}" rpy="0 0 0"/>
-        </xacro:inertial_cylinder>
-    </link>
-    <gazebo reference="lf_wheel">
-        <material>Gazebo/Red</material>
-    </gazebo>
-    <!-- RIGHT FRONT WHEEL LINK -->
-    <joint name="rf_wheel_joint" type="continuous">
-        <parent link="front_chassis"/>
-        <child link="rf_wheel"/>
-        <origin xyz="${scaled_wheel_length / 2 - scaled_wheel_radius / 2} -${scaled_chassis_radius} 0" rpy="${pi/2} 0 0"/>
-        <axis xyz="0 0 -1"/>
-    </joint>
-    <link name="rf_wheel">
-        <visual>
-            <origin xyz="0 0 ${scaled_wheel_length / 2}" rpy="0 0 0"/>
-            <geometry>
-                <cylinder radius="${scaled_wheel_radius}" length="${scaled_wheel_length}"/>
-            </geometry>
-            <material name="red"/>
-        </visual>
-        <collision>
-            <origin xyz="0 0 ${scaled_wheel_length / 2}" rpy="0 0 0"/>
-            <geometry>
-                <cylinder radius="${scaled_wheel_radius}" length="${scaled_wheel_length}"/>
-            </geometry>
-        </collision>
-        <xacro:inertial_cylinder mass="${scaled_wheel_mass}" radius="${scaled_wheel_radius}" length="${scaled_wheel_length}">
-            <origin xyz="0 0 ${scaled_wheel_length / 2}" rpy="0 0 0"/>
-        </xacro:inertial_cylinder>
-    </link>
-    <gazebo reference="rf_wheel">
-        <material>Gazebo/Red</material>
-    </gazebo>
-    <!-- FRONT CASTER WHEEL LINK -->
-    <joint name="f_caster_wheel_joint" type="fixed">
-        <parent link="front_chassis"/>
-        <child link="f_caster_wheel"/>
-        <origin xyz="${scaled_chassis_length / 4} 0 -${scaled_wheel_radius / 2}" rpy="0 0 0"/>
-    </joint>
-    <link name="f_caster_wheel">
-        <visual>
-            <geometry>
-                <sphere radius="${scaled_wheel_radius / 2}"/>
-            </geometry>
-            <material name="black"/>
-        </visual>
-        <collision>
-            <geometry>
-                <sphere radius="${scaled_wheel_radius / 2}"/>
-            </geometry>
-        </collision>
-        <xacro:inertial_sphere mass="${scaled_caster_wheel_mass}" radius="${scaled_wheel_radius / 2}">
-            <origin xyz="0 0 0" rpy="0 0 0"/>
-        </xacro:inertial_sphere>
-    </link>
-    <gazebo reference="f_caster_wheel">
+    <gazebo reference="caster_wheel">
         <material>Gazebo/Black</material>
         <mu1 value="0.001"/>
@@ -267,5 +155,5 @@
     <!-- CAMERA -->
     <joint name="camera_joint" type="fixed">
-        <parent link="front_chassis"/>
+        <parent link="chassis"/>
         <child link="camera_link"/>
         <origin xyz="${scaled_chassis_length / 2} 0 0" rpy="0 0 0"/>
