Commit message: 0331

File: urdf/robot_core_1.xacro (robot description, xacro)
@@ -32,5 +32,5 @@
     <xacro:property name="chassis_mass" value="0.002"/>
     <xacro:property name="wheel_mass" value="0.001"/>
-    <xacro:property name="caster_wheel_mass" value="0.001"/>
+    <xacro:property name="caster_wheel_mass" value="0.01"/>
     <!-- Update All Parameters from a Single Parameter -->
     <xacro:property name="scale" value="50.0"/>
@@ -43,11 +43,11 @@
     <xacro:property name="scaled_caster_wheel_mass" value="${caster_wheel_mass * scale}"/>
     <xacro:property name="scaled_camera_length" value="${scaled_chassis_radius / 5}"/>
-    <!-- BACK CHASSIS LINK -->
-    <joint name="back_chassis_joint" type="fixed">
+    <!-- CHASSIS LINK -->
+    <joint name="chassis_joint" type="fixed">
         <parent link="base_link"/>
-        <child link="back_chassis"/>
+        <child link="chassis"/>
         <origin xyz="${scaled_chassis_length / 2} 0 ${scaled_wheel_radius}" rpy="0 0 0"/>
     </joint>
-    <link name="back_chassis">
+    <link name="chassis">
         <visual>
             <origin xyz="0 0 0" rpy="0 ${pi/2} 0"/>
@@ -60,5 +60,5 @@
             <origin xyz="0 0 0" rpy="0 ${pi/2} 0"/>
             <geometry>
-                <cylinder radius="${scaled_chassis_radius}" length="${scaled_chassis_length * 0.8}"/>
+                <cylinder radius="${scaled_chassis_radius}" length="${scaled_chassis_length}"/>
             </geometry>
         </collision>
@@ -67,15 +67,15 @@
         </xacro:inertial_cylinder>
     </link>
-    <gazebo reference="back_chassis">
+    <gazebo reference="chassis">
         <material>Gazebo/White</material>
     </gazebo>
-    <!-- LEFT BACK WHEEL LINK -->
-    <joint name="lb_wheel_joint" type="continuous">
+    <!-- LEFT WHEEL LINK -->
+    <joint name="left_wheel_joint" type="continuous">
         <parent link="base_link"/>
-        <child link="lb_wheel"/>
+        <child link="left_wheel"/>
         <origin xyz="${scaled_wheel_radius} ${scaled_chassis_radius} ${scaled_wheel_radius}" rpy="-${pi/2} 0 0" />
         <axis xyz="0 0 1"/>
     </joint>
-    <link name="lb_wheel">
+    <link name="left_wheel">
         <visual>
             <origin xyz="0 0 ${scaled_wheel_length / 2}" rpy="0 0 0"/>
@@ -95,15 +95,15 @@
         </xacro:inertial_cylinder>
     </link>
-    <gazebo reference="lb_wheel">
+    <gazebo reference="left_wheel">
         <material>Gazebo/Blue</material>
     </gazebo>
-    <!-- RIGHT BACK WHEEL LINK -->
-    <joint name="rb_wheel_joint" type="continuous">
+    <!-- RIGHT WHEEL LINK -->
+    <joint name="right_wheel_joint" type="continuous">
         <parent link="base_link"/>
-        <child link="rb_wheel"/>
+        <child link="right_wheel"/>
         <origin xyz="${scaled_wheel_radius} -${scaled_chassis_radius} ${scaled_wheel_radius}" rpy="${pi/2} 0 0" />
         <axis xyz="0 0 -1"/>
     </joint>
-    <link name="rb_wheel">
+    <link name="right_wheel">
         <visual>
             <origin xyz="0 0 ${scaled_wheel_length / 2}" rpy="0 0 0"/>
@@ -123,14 +123,14 @@
         </xacro:inertial_cylinder>
     </link>
-    <gazebo reference="rb_wheel">
+    <gazebo reference="right_wheel">
         <material>Gazebo/Blue</material>
     </gazebo>
-    <!-- BACK CASTER WHEEL LINK -->
-    <joint name="b_caster_wheel_joint" type="fixed">
-        <parent link="back_chassis"/>
-        <child link="b_caster_wheel"/>
+    <!-- CASTER WHEEL LINK -->
+    <joint name="caster_wheel_joint" type="fixed">
+        <parent link="chassis"/>
+        <child link="caster_wheel"/>
         <origin xyz="${scaled_chassis_length / 4} 0 -${scaled_wheel_radius / 2}" rpy="0 0 0"/>
     </joint>
-    <link name="b_caster_wheel">
+    <link name="caster_wheel">
         <visual>
             <geometry>
@@ -148,136 +148,5 @@
         </xacro:inertial_sphere>
     </link>
-    <gazebo reference="b_caster_wheel">
-        <material>Gazebo/Black</material>
-        <mu1 value="0.001"/>
-        <mu2 value="0.001"/>
-    </gazebo>
-    <!-- FRONT CHASSIS LINK -->
-    <joint name="roll_joint" type="revolute">
-        <parent link="back_chassis"/>
-        <child link="roll_link"/>
-        <origin xyz="${scaled_chassis_length / 2} 0 0" rpy="0 0 0"/>
-        <axis xyz="1 0 0"/>
-        <limit velocity="10.0" effort="200" lower="-${pi}" upper="${pi}"/>
-    </joint>
-    <!-- Roll Joint -->
-    <link name="roll_link"/>
-    <!-- Pitch Joint -->
-    <joint name="pitch_joint" type="revolute">
-        <parent link="roll_link"/>
-        <child link="pitch_link"/>
-        <origin xyz="0 0 0" rpy="0 0 0"/>
-        <axis xyz="0 1 0"/>
-        <limit velocity="10.0" effort="200" lower="-${pi}" upper="${pi}"/>
-    </joint>
-    <link name="pitch_link"/>
-    <!-- Yaw Joint -->
-    <joint name="yaw_joint" type="revolute">
-        <parent link="pitch_link"/>
-        <child link="front_chassis"/>
-        <origin xyz="0 0 0" rpy="0 0 0"/>
-        <axis xyz="0 0 1"/>
-        <limit velocity="10.0" effort="200" lower="-${pi}" upper="${pi}"/>
-    </joint>
-    <link name="front_chassis">
-        <visual>
-            <origin xyz="${scaled_chassis_length / 2} 0 0" rpy="0 ${pi/2} 0"/>
-            <geometry>
-                <cylinder radius="${scaled_chassis_radius}" length="${scaled_chassis_length}"/>
-            </geometry>
-            <material name="white"/>
-        </visual>
-        <collision>
-            <origin xyz="${scaled_chassis_length / 2} 0 0" rpy="0 ${pi/2} 0"/>
-            <geometry>
-                <cylinder radius="${scaled_chassis_radius}" length="${scaled_chassis_length * 0.8}"/>
-            </geometry>
-        </collision>
-        <xacro:inertial_cylinder mass="${scaled_chassis_mass}" radius="${scaled_chassis_radius}" length="${scaled_chassis_length}">
-            <origin xyz="${scaled_chassis_length / 2} 0 0" rpy="0 ${pi/2} 0"/>
-        </xacro:inertial_cylinder>
-    </link>
-    <gazebo reference="front_chassis">
-        <material>Gazebo/White</material>
-    </gazebo>
-    <!-- LEFT FRONT WHEEL LINK -->
-    <joint name="lf_wheel_joint" type="continuous">
-        <parent link="front_chassis"/>
-        <child link="lf_wheel"/>
-        <origin xyz="${scaled_wheel_radius} ${scaled_chassis_radius} 0" rpy="-${pi/2} 0 0"/>
-        <axis xyz="0 0 1"/>
-    </joint>
-    <link name="lf_wheel">
-        <visual>
-            <origin xyz="0 0 ${scaled_wheel_length / 2}" rpy="0 0 0"/>
-            <geometry>
-                <cylinder radius="${scaled_wheel_radius}" length="${scaled_wheel_length}"/>
-            </geometry>
-            <material name="red"/>
-        </visual>
-        <collision>
-            <origin xyz="0 0 ${scaled_wheel_length / 2}" rpy="0 0 0"/>
-            <geometry>
-                <cylinder radius="${scaled_wheel_radius}" length="${scaled_wheel_length}"/>
-            </geometry>
-        </collision>
-        <xacro:inertial_cylinder mass="${scaled_wheel_mass}" radius="${scaled_wheel_radius}" length="${scaled_wheel_length}">
-            <origin xyz="0 0 ${scaled_wheel_length / 2}" rpy="0 0 0"/>
-        </xacro:inertial_cylinder>
-    </link>
-    <gazebo reference="lf_wheel">
-        <material>Gazebo/Red</material>
-    </gazebo>
-    <!-- RIGHT FRONT WHEEL LINK -->
-    <joint name="rf_wheel_joint" type="continuous">
-        <parent link="front_chassis"/>
-        <child link="rf_wheel"/>
-        <origin xyz="${scaled_wheel_radius} -${scaled_chassis_radius} 0" rpy="${pi/2} 0 0"/>
-        <axis xyz="0 0 -1"/>
-    </joint>
-    <link name="rf_wheel">
-        <visual>
-            <origin xyz="0 0 ${scaled_wheel_length / 2}" rpy="0 0 0"/>
-            <geometry>
-                <cylinder radius="${scaled_wheel_radius}" length="${scaled_wheel_length}"/>
-            </geometry>
-            <material name="red"/>
-        </visual>
-        <collision>
-            <origin xyz="0 0 ${scaled_wheel_length / 2}" rpy="0 0 0"/>
-            <geometry>
-                <cylinder radius="${scaled_wheel_radius}" length="${scaled_wheel_length}"/>
-            </geometry>
-        </collision>
-        <xacro:inertial_cylinder mass="${scaled_wheel_mass}" radius="${scaled_wheel_radius}" length="${scaled_wheel_length}">
-            <origin xyz="0 0 ${scaled_wheel_length / 2}" rpy="0 0 0"/>
-        </xacro:inertial_cylinder>
-    </link>
-    <gazebo reference="rf_wheel">
-        <material>Gazebo/Red</material>
-    </gazebo>
-    <!-- FRONT CASTER WHEEL LINK -->
-    <joint name="f_caster_wheel_joint" type="fixed">
-        <parent link="front_chassis"/>
-        <child link="f_caster_wheel"/>
-        <origin xyz="${scaled_chassis_length / 4} 0 -${scaled_wheel_radius / 2}" rpy="0 0 0"/>
-    </joint>
-    <link name="f_caster_wheel">
-        <visual>
-            <geometry>
-                <sphere radius="${scaled_wheel_radius / 2}"/>
-            </geometry>
-            <material name="black"/>
-        </visual>
-        <collision>
-            <geometry>
-                <sphere radius="${scaled_wheel_radius / 2}"/>
-            </geometry>
-        </collision>
-        <xacro:inertial_sphere mass="${scaled_caster_wheel_mass}" radius="${scaled_wheel_radius / 2}">
-            <origin xyz="0 0 0" rpy="0 0 0"/>
-        </xacro:inertial_sphere>
-    </link>
-    <gazebo reference="f_caster_wheel">
+    <gazebo reference="caster_wheel">
         <material>Gazebo/Black</material>
         <mu1 value="0.001"/>
@@ -286,5 +155,5 @@
     <!-- CAMERA -->
     <joint name="camera_joint" type="fixed">
-        <parent link="front_chassis"/>
+        <parent link="chassis"/>
         <child link="camera_link"/>
         <origin xyz="${scaled_chassis_length / 2} 0 0" rpy="0 0 0"/>

File: urdf/robot_core_2.xacro (robot description, xacro)
@@ -6,5 +6,4 @@
     <!-- <xacro:include filename="depth_camera.xacro"/> -->
     <xacro:include filename="rgb_camera.xacro"/>
-    <!-- <xacro:include filename="gazebo_control.xacro"/> -->
     <!-- COLORS -->
     <material name="white">
@@ -153,30 +152,11 @@
         <mu2 value="0.001"/>
     </gazebo>
-    <!-- FRONT CHASSIS LINK -->
-    <joint name="roll_joint" type="revolute">
+    <!-- CHASSIS BETWEEN JOINT -->
+    <joint name="joint_between_chassis" type="revolute">
         <parent link="back_chassis"/>
-        <child link="roll_link"/>
-        <origin xyz="${scaled_chassis_length / 2} 0 0" rpy="0 0 0"/>
-        <axis xyz="1 0 0"/>
-        <limit velocity="10.0" effort="200" lower="-${pi}" upper="${pi}"/>
-    </joint>
-    <!-- Roll Joint -->
-    <link name="roll_link"/>
-    <!-- Pitch Joint -->
-    <joint name="pitch_joint" type="revolute">
-        <parent link="roll_link"/>
-        <child link="pitch_link"/>
-        <origin xyz="0 0 0" rpy="0 0 0"/>
-        <axis xyz="0 1 0"/>
-        <limit velocity="10.0" effort="200" lower="-${pi}" upper="${pi}"/>
-    </joint>
-    <link name="pitch_link"/>
-    <!-- Yaw Joint -->
-    <joint name="yaw_joint" type="revolute">
-        <parent link="pitch_link"/>
         <child link="front_chassis"/>
-        <origin xyz="0 0 0" rpy="0 0 0"/>
+        <origin xyz="${scaled_chassis_length / 2}  0 0" rpy="0 0 0"/>
         <axis xyz="0 0 1"/>
-        <limit velocity="10.0" effort="200" lower="-${pi}" upper="${pi}"/>
+        <limit effort="200.0" lower="${-pi/2}" upper="${pi/2}" velocity="1.0"/>
     </joint>
     <link name="front_chassis">
@@ -284,4 +264,11 @@
         <mu2 value="0.001"/>
     </gazebo>
+    <!-- <gazebo>
+        <plugin name="gazebo_ros2_control" filename="libgazebo_ros2_control.so">
+            <ros2_control_plugin>gazebo_ros2_control/GazeboSystem</ros2_control_plugin>
+            <control_period>0.001</control_period>
+            <parameters>$(find endoscope)/config/ros2_control.yaml</parameters>
+        </plugin>
+    </gazebo> -->
     <!-- CAMERA -->
     <joint name="camera_joint" type="fixed">

File: urdf/robot_exe.xacro (robot description, xacro)
@@ -1,5 +1,6 @@
 <?xml version="1.0"?>
 <robot xmlns:xacro="http://www.ros.org/wiki/xacro" name="endoscope">
-    <xacro:include filename="robot_core.xacro"/>
-    <xacro:include filename="gazebo_control.xacro"/>
+    <xacro:include filename="robot_core_2.xacro"/>
+    <!-- <xacro:include filename="keyboard_control.xacro"/> -->
+    <xacro:include filename="joystick_control.xacro"/>
 </robot>
