Commit message: 0402

File: description/keyboard_control.xacro (robot description, xacro)
@@ -3,4 +3,7 @@
     <gazebo>
         <plugin name="diff_drive" filename="libgazebo_ros_diff_drive.so">
+            <ros>
+                <remapping>cmd_vel:=cmd_vel_straight</remapping>
+            </ros>
             <!-- Wheel Information -->
             <left_joint>lb_wheel_joint</left_joint>
@@ -8,11 +11,8 @@
             <wheel_separation>${2 * scaled_chassis_radius + scaled_wheel_length}</wheel_separation>
             <wheel_diameter>${2 * scaled_wheel_radius}</wheel_diameter>
-            <!-- <wheel_separation>0.35</wheel_separation>
-            <wheel_diameter>0.1</wheel_diameter> -->
             <!-- Limits -->
             <max_wheel_torque>200</max_wheel_torque>
             <max_wheel_acceleration>10.0</max_wheel_acceleration>
             <!-- Output -->
-            <command_topic>cmd_vel</command_topic>
             <odometry_frame>odom</odometry_frame>
             <robot_base_frame>base_link</robot_base_frame>

File: description/robot_core.xacro (robot description, xacro)
@@ -6,5 +6,4 @@
     <!-- <xacro:include filename="depth_camera.xacro"/> -->
     <xacro:include filename="rgb_camera.xacro"/>
-    <!-- <xacro:include filename="gazebo_control.xacro"/> -->
     <!-- COLORS -->
     <material name="white">
@@ -27,10 +26,10 @@
     <!-- DEFINE PARAMETERS -->
     <xacro:property name="chassis_radius" value="0.0065"/>
-    <xacro:property name="chassis_length" value="0.02"/>
+    <xacro:property name="chassis_length" value="0.03"/>
     <xacro:property name="wheel_radius" value="0.008"/>
     <xacro:property name="wheel_length" value="0.001"/>
-    <xacro:property name="chassis_mass" value="0.002"/>
-    <xacro:property name="wheel_mass" value="0.001"/>
-    <xacro:property name="caster_wheel_mass" value="0.01"/>
+    <xacro:property name="chassis_mass" value="0.001"/>
+    <xacro:property name="wheel_mass" value="0.0005"/>
+    <xacro:property name="caster_wheel_mass" value="0.0005"/>
     <!-- Update All Parameters from a Single Parameter -->
     <xacro:property name="scale" value="50.0"/>
@@ -43,11 +42,11 @@
     <xacro:property name="scaled_caster_wheel_mass" value="${caster_wheel_mass * scale}"/>
     <xacro:property name="scaled_camera_length" value="${scaled_chassis_radius / 5}"/>
-    <!-- CHASSIS LINK -->
-    <joint name="chassis_joint" type="fixed">
+    <!-- BACK CHASSIS LINK -->
+    <joint name="back_chassis_joint" type="fixed">
         <parent link="base_link"/>
-        <child link="chassis"/>
+        <child link="back_chassis"/>
         <origin xyz="${scaled_chassis_length / 2} 0 ${scaled_wheel_radius}" rpy="0 0 0"/>
     </joint>
-    <link name="chassis">
+    <link name="back_chassis">
         <visual>
             <origin xyz="0 0 0" rpy="0 ${pi/2} 0"/>
@@ -60,5 +59,5 @@
             <origin xyz="0 0 0" rpy="0 ${pi/2} 0"/>
             <geometry>
-                <cylinder radius="${scaled_chassis_radius}" length="${scaled_chassis_length}"/>
+                <cylinder radius="${scaled_chassis_radius * 0.8}" length="${scaled_chassis_length * 0.8}"/>
             </geometry>
         </collision>
@@ -67,15 +66,15 @@
         </xacro:inertial_cylinder>
     </link>
-    <gazebo reference="chassis">
+    <gazebo reference="back_chassis">
         <material>Gazebo/White</material>
     </gazebo>
-    <!-- LEFT WHEEL LINK -->
-    <joint name="left_wheel_joint" type="continuous">
+    <!-- LEFT BACK WHEEL LINK -->
+    <joint name="lb_wheel_joint" type="continuous">
         <parent link="base_link"/>
-        <child link="left_wheel"/>
+        <child link="lb_wheel"/>
         <origin xyz="${scaled_wheel_radius} ${scaled_chassis_radius} ${scaled_wheel_radius}" rpy="-${pi/2} 0 0" />
         <axis xyz="0 0 1"/>
     </joint>
-    <link name="left_wheel">
+    <link name="lb_wheel">
         <visual>
             <origin xyz="0 0 ${scaled_wheel_length / 2}" rpy="0 0 0"/>
@@ -95,15 +94,15 @@
         </xacro:inertial_cylinder>
     </link>
-    <gazebo reference="left_wheel">
+    <gazebo reference="lb_wheel">
         <material>Gazebo/Blue</material>
     </gazebo>
-    <!-- RIGHT WHEEL LINK -->
-    <joint name="right_wheel_joint" type="continuous">
+    <!-- RIGHT BACK WHEEL LINK -->
+    <joint name="rb_wheel_joint" type="continuous">
         <parent link="base_link"/>
-        <child link="right_wheel"/>
+        <child link="rb_wheel"/>
         <origin xyz="${scaled_wheel_radius} -${scaled_chassis_radius} ${scaled_wheel_radius}" rpy="${pi/2} 0 0" />
         <axis xyz="0 0 -1"/>
     </joint>
-    <link name="right_wheel">
+    <link name="rb_wheel">
         <visual>
             <origin xyz="0 0 ${scaled_wheel_length / 2}" rpy="0 0 0"/>
@@ -123,14 +122,14 @@
         </xacro:inertial_cylinder>
     </link>
-    <gazebo reference="right_wheel">
+    <gazebo reference="rb_wheel">
         <material>Gazebo/Blue</material>
     </gazebo>
-    <!-- CASTER WHEEL LINK -->
-    <joint name="caster_wheel_joint" type="fixed">
-        <parent link="chassis"/>
-        <child link="caster_wheel"/>
+    <!-- BACK CASTER WHEEL LINK -->
+    <joint name="b_caster_wheel_joint" type="fixed">
+        <parent link="back_chassis"/>
+        <child link="b_caster_wheel"/>
         <origin xyz="${scaled_chassis_length / 4} 0 -${scaled_wheel_radius / 2}" rpy="0 0 0"/>
     </joint>
-    <link name="caster_wheel">
+    <link name="b_caster_wheel">
         <visual>
             <geometry>
@@ -148,14 +147,126 @@
         </xacro:inertial_sphere>
     </link>
-    <gazebo reference="caster_wheel">
+    <gazebo reference="b_caster_wheel">
         <material>Gazebo/Black</material>
         <mu1 value="0.001"/>
         <mu2 value="0.001"/>
     </gazebo>
+    <!-- CHASSIS BETWEEN JOINT -->
+    <joint name="joint_between_chassis" type="revolute">
+        <parent link="back_chassis"/>
+        <child link="front_chassis"/>
+        <origin xyz="${scaled_chassis_length / 2}  0 0" rpy="0 0 0"/>
+        <axis xyz="0 0 1"/>
+        <limit effort="200.0" lower="${-pi/3}" upper="${pi/3}" velocity="1.0"/>
+    </joint>
+    <link name="front_chassis">
+        <visual>
+            <origin xyz="${scaled_chassis_length / 2} 0 0" rpy="0 ${pi/2} 0"/>
+            <geometry>
+                <cylinder radius="${scaled_chassis_radius}" length="${scaled_chassis_length}"/>
+            </geometry>
+            <material name="white"/>
+        </visual>
+        <collision>
+            <origin xyz="${scaled_chassis_length / 2} 0 0" rpy="0 ${pi/2} 0"/>
+            <geometry>
+                <cylinder radius="${scaled_chassis_radius * 0.8}" length="${scaled_chassis_length * 0.8}"/>
+            </geometry>
+        </collision>
+        <xacro:inertial_cylinder mass="${scaled_chassis_mass}" radius="${scaled_chassis_radius}" length="${scaled_chassis_length}">
+            <origin xyz="${scaled_chassis_length / 2} 0 0" rpy="0 ${pi/2} 0"/>
+        </xacro:inertial_cylinder>
+    </link>
+    <gazebo reference="front_chassis">
+        <material>Gazebo/White</material>
+    </gazebo>
+    <!-- LEFT FRONT WHEEL LINK -->
+    <joint name="lf_wheel_joint" type="continuous">
+        <parent link="front_chassis"/>
+        <child link="lf_wheel"/>
+        <origin xyz="${scaled_wheel_radius} ${scaled_chassis_radius} 0" rpy="-${pi/2} 0 0"/>
+        <axis xyz="0 0 1"/>
+    </joint>
+    <link name="lf_wheel">
+        <visual>
+            <origin xyz="0 0 ${scaled_wheel_length / 2}" rpy="0 0 0"/>
+            <geometry>
+                <cylinder radius="${scaled_wheel_radius}" length="${scaled_wheel_length}"/>
+            </geometry>
+            <material name="red"/>
+        </visual>
+        <collision>
+            <origin xyz="0 0 ${scaled_wheel_length / 2}" rpy="0 0 0"/>
+            <geometry>
+                <cylinder radius="${scaled_wheel_radius}" length="${scaled_wheel_length}"/>
+            </geometry>
+        </collision>
+        <xacro:inertial_cylinder mass="${scaled_wheel_mass}" radius="${scaled_wheel_radius}" length="${scaled_wheel_length}">
+            <origin xyz="0 0 ${scaled_wheel_length / 2}" rpy="0 0 0"/>
+        </xacro:inertial_cylinder>
+    </link>
+    <gazebo reference="lf_wheel">
+        <material>Gazebo/Red</material>
+    </gazebo>
+    <!-- RIGHT FRONT WHEEL LINK -->
+    <joint name="rf_wheel_joint" type="continuous">
+        <parent link="front_chassis"/>
+        <child link="rf_wheel"/>
+        <origin xyz="${scaled_wheel_radius} -${scaled_chassis_radius} 0" rpy="${pi/2} 0 0"/>
+        <axis xyz="0 0 -1"/>
+    </joint>
+    <link name="rf_wheel">
+        <visual>
+            <origin xyz="0 0 ${scaled_wheel_length / 2}" rpy="0 0 0"/>
+            <geometry>
+                <cylinder radius="${scaled_wheel_radius}" length="${scaled_wheel_length}"/>
+            </geometry>
+            <material name="red"/>
+        </visual>
+        <collision>
+            <origin xyz="0 0 ${scaled_wheel_length / 2}" rpy="0 0 0"/>
+            <geometry>
+                <cylinder radius="${scaled_wheel_radius}" length="${scaled_wheel_length}"/>
+            </geometry>
+        </collision>
+        <xacro:inertial_cylinder mass="${scaled_wheel_mass}" radius="${scaled_wheel_radius}" length="${scaled_wheel_length}">
+            <origin xyz="0 0 ${scaled_wheel_length / 2}" rpy="0 0 0"/>
+        </xacro:inertial_cylinder>
+    </link>
+    <gazebo reference="rf_wheel">
+        <material>Gazebo/Red</material>
+    </gazebo>
+    <!-- FRONT CASTER WHEEL LINK -->
+    <joint name="f_caster_wheel_joint" type="fixed">
+        <parent link="front_chassis"/>
+        <child link="f_caster_wheel"/>
+        <origin xyz="${scaled_chassis_length * 0.75} 0 -${scaled_wheel_radius / 2}" rpy="0 0 0"/>
+    </joint>
+    <link name="f_caster_wheel">
+        <visual>
+            <geometry>
+                <sphere radius="${scaled_wheel_radius / 2}"/>
+            </geometry>
+            <material name="black"/>
+        </visual>
+        <collision>
+            <geometry>
+                <sphere radius="${scaled_wheel_radius / 2}"/>
+            </geometry>
+        </collision>
+        <xacro:inertial_sphere mass="${scaled_caster_wheel_mass}" radius="${scaled_wheel_radius / 2}">
+            <origin xyz="0 0 0" rpy="0 0 0"/>
+        </xacro:inertial_sphere>
+    </link>
+    <gazebo reference="f_caster_wheel">
+        <material>Gazebo/Black</material>
+        <mu1 value="0.001"/>
+        <mu2 value="0.001"/>
+    </gazebo>
     <!-- CAMERA -->
     <joint name="camera_joint" type="fixed">
-        <parent link="chassis"/>
+        <parent link="front_chassis"/>
         <child link="camera_link"/>
-        <origin xyz="${scaled_chassis_length / 2} 0 0" rpy="0 0 0"/>
+        <origin xyz="${scaled_chassis_length} 0 0" rpy="0 0 0"/>
     </joint>
     <link name="camera_link">

File: description/robot_core_test.xacro (robot description, xacro)
@@ -1,9 +1,4 @@
 <?xml version="1.0"?>
 <robot xmlns:xacro="http://www.ros.org/wiki/xacro" >
-    <!-- INERTIAL SETTINGS -->
-    <xacro:include filename="inertial_macros.xacro"/>
-    <!-- CAMERA PARAMETERS -->
-    <!-- <xacro:include filename="depth_camera.xacro"/> -->
-    <xacro:include filename="rgb_camera.xacro"/>
     <!-- COLORS -->
     <material name="white">
@@ -26,10 +21,10 @@
     <!-- DEFINE PARAMETERS -->
     <xacro:property name="chassis_radius" value="0.0065"/>
-    <xacro:property name="chassis_length" value="0.02"/>
+    <xacro:property name="chassis_length" value="0.03"/>
     <xacro:property name="wheel_radius" value="0.008"/>
     <xacro:property name="wheel_length" value="0.001"/>
-    <xacro:property name="chassis_mass" value="0.002"/>
-    <xacro:property name="wheel_mass" value="0.001"/>
-    <xacro:property name="caster_wheel_mass" value="0.001"/>
+    <xacro:property name="chassis_mass" value="0.001"/>
+    <xacro:property name="wheel_mass" value="0.0005"/>
+    <xacro:property name="caster_wheel_mass" value="0.0005"/>
     <!-- Update All Parameters from a Single Parameter -->
     <xacro:property name="scale" value="50.0"/>
@@ -59,5 +54,5 @@
             <origin xyz="0 0 0" rpy="0 ${pi/2} 0"/>
             <geometry>
-                <cylinder radius="${scaled_chassis_radius}" length="${scaled_chassis_length * 0.8}"/>
+                <cylinder radius="${scaled_chassis_radius * 0.8}" length="${scaled_chassis_length * 0.8}"/>
             </geometry>
         </collision>
@@ -158,5 +153,5 @@
         <origin xyz="${scaled_chassis_length / 2}  0 0" rpy="0 0 0"/>
         <axis xyz="0 0 1"/>
-        <limit effort="200.0" lower="${-pi/2}" upper="${pi/2}" velocity="1.0"/>
+        <limit effort="200.0" lower="${-pi/4}" upper="${pi/4}" velocity="1.0"/>
     </joint>
     <link name="front_chassis">
@@ -164,5 +159,5 @@
             <origin xyz="${scaled_chassis_length / 2} 0 0" rpy="0 ${pi/2} 0"/>
             <geometry>
-                <cylinder radius="${scaled_chassis_radius}" length="${scaled_chassis_length}"/>
+                <cylinder radius="${scaled_chassis_radius / 2}" length="${scaled_chassis_length}"/>
             </geometry>
             <material name="white"/>
@@ -171,5 +166,5 @@
             <origin xyz="${scaled_chassis_length / 2} 0 0" rpy="0 ${pi/2} 0"/>
             <geometry>
-                <cylinder radius="${scaled_chassis_radius}" length="${scaled_chassis_length * 0.8}"/>
+                <cylinder radius="${scaled_chassis_radius * 0.8}" length="${scaled_chassis_length * 0.8}"/>
             </geometry>
         </collision>
@@ -241,5 +236,5 @@
         <parent link="front_chassis"/>
         <child link="f_caster_wheel"/>
-        <origin xyz="${scaled_chassis_length / 4} 0 -${scaled_wheel_radius / 2}" rpy="0 0 0"/>
+        <origin xyz="${scaled_chassis_length * 0.75} 0 -${scaled_wheel_radius / 2}" rpy="0 0 0"/>
     </joint>
     <link name="f_caster_wheel">
@@ -264,16 +259,9 @@
         <mu2 value="0.001"/>
     </gazebo>
-    <!-- <gazebo>
-        <plugin name="gazebo_ros2_control" filename="libgazebo_ros2_control.so">
-            <ros2_control_plugin>gazebo_ros2_control/GazeboSystem</ros2_control_plugin>
-            <control_period>0.001</control_period>
-            <parameters>$(find endoscope)/config/ros2_control.yaml</parameters>
-        </plugin>
-    </gazebo> -->
     <!-- CAMERA -->
     <joint name="camera_joint" type="fixed">
         <parent link="front_chassis"/>
         <child link="camera_link"/>
-        <origin xyz="${scaled_chassis_length / 2} 0 0" rpy="0 0 0"/>
+        <origin xyz="${scaled_chassis_length} 0 0" rpy="0 0 0"/>
     </joint>
     <link name="camera_link">
