Commit message: 0402

File: description/control.xacro (robot description, xacro)
@@ -5,8 +5,44 @@
             <plugin>gazebo_ros2_control/GazeboSystem</plugin>
         </hardware>
-        <joint name="joint_between_chassis">
+        <joint name="lb_wheel_joint">
             <command_interface name="velocity">
-                <param name="min">-10</param>
-                <param name="max">10</param>
+                <param name="min">-1</param>
+                <param name="max">1</param>
+            </command_interface>
+            <state_interface name="position"/>
+            <state_interface name="velocity"/>
+            <state_interface name="effort"/>
+        </joint>
+        <joint name="rb_wheel_joint">
+            <command_interface name="velocity">
+                <param name="min">-1</param>
+                <param name="max">1</param>
+            </command_interface>
+            <state_interface name="position"/>
+            <state_interface name="velocity"/>
+            <state_interface name="effort"/>
+        </joint>
+        <joint name="front_chassis_roll_joint">
+            <command_interface name="position">
+                <param name="min">-1</param>
+                <param name="max">1</param>
+            </command_interface>
+            <state_interface name="position"/>
+            <state_interface name="velocity"/>
+            <state_interface name="effort"/>
+        </joint>
+        <joint name="front_chassis_pitch_joint">
+            <command_interface name="position">
+                <param name="min">-1</param>
+                <param name="max">1</param>
+            </command_interface>
+            <state_interface name="position"/>
+            <state_interface name="velocity"/>
+            <state_interface name="effort"/>
+        </joint>
+        <joint name="front_chassis_yaw_joint">
+            <command_interface name="position">
+                <param name="min">-1</param>
+                <param name="max">1</param>
             </command_interface>
             <state_interface name="position"/>

File: description/keyboard_control.xacro (robot description, xacro)
@@ -4,5 +4,5 @@
         <plugin name="diff_drive" filename="libgazebo_ros_diff_drive.so">
             <ros>
-                <remapping>cmd_vel:=cmd_vel_straight</remapping>
+                <remapping>cmd_vel:=cmd_vel</remapping>
             </ros>
             <!-- Wheel Information -->

File: description/robot_core.xacro (robot description, xacro)
@@ -1,9 +1,4 @@
 <?xml version="1.0"?>
-<robot xmlns:xacro="http://www.ros.org/wiki/xacro" >
-    <!-- INERTIAL SETTINGS -->
-    <xacro:include filename="inertial_macros.xacro"/>
-    <!-- CAMERA PARAMETERS -->
-    <!-- <xacro:include filename="depth_camera.xacro"/> -->
-    <xacro:include filename="rgb_camera.xacro"/>
+<robot xmlns:xacro="http://www.ros.org/wiki/xacro" name="colonoscopy">
     <!-- COLORS -->
     <material name="white">
@@ -29,7 +24,7 @@
     <xacro:property name="wheel_radius" value="0.008"/>
     <xacro:property name="wheel_length" value="0.001"/>
-    <xacro:property name="chassis_mass" value="0.001"/>
-    <xacro:property name="wheel_mass" value="0.0005"/>
-    <xacro:property name="caster_wheel_mass" value="0.0005"/>
+    <xacro:property name="chassis_mass" value="1.0"/>
+    <xacro:property name="wheel_mass" value="0.005"/>
+    <xacro:property name="caster_wheel_mass" value="0.005"/>
     <!-- Update All Parameters from a Single Parameter -->
     <xacro:property name="scale" value="50.0"/>
@@ -153,10 +148,39 @@
     </gazebo>
     <!-- CHASSIS BETWEEN JOINT -->
-    <joint name="joint_between_chassis" type="revolute">
+    <joint name="front_chassis_roll_joint" type="revolute">
         <parent link="back_chassis"/>
+        <child link="front_chassis_roll_link"/>
+        <origin xyz="${scaled_chassis_length / 2}  0 0" rpy="0 0 0"/>
+        <axis xyz="1 0 0"/>
+        <limit lower="-0.5" upper="0.5" effort="1000.0" velocity="1.0"/>
+        <dynamics damping="1.0" friction="0.1"/>
+    </joint>
+    <link name="front_chassis_roll_link">
+        <inertial>
+            <mass value="0.001"/>
+            <inertia ixx="1e-6" ixy="0" ixz="0" iyy="1e-6" iyz="0" izz="1e-6"/>
+        </inertial>
+    </link>
+    <!-- Pitch Joint -->
+    <joint name="front_chassis_pitch_joint" type="revolute">
+        <parent link="front_chassis_roll_link"/>
+        <child link="front_chassis_pitch_link"/>
+        <axis xyz="0 1 0"/>
+        <origin xyz="0 0 0" rpy="0 0 0"/>
+        <limit lower="-0.5" upper="0.5" effort="1000" velocity="1.0"/>
+    </joint>
+    <link name="front_chassis_pitch_link">
+        <inertial>
+            <mass value="0.001"/>
+            <inertia ixx="1e-6" ixy="0" ixz="0" iyy="1e-6" iyz="0" izz="1e-6"/>
+        </inertial>
+    </link>
+    <!-- Yaw Joint -->
+    <joint name="front_chassis_yaw_joint" type="revolute">
+        <parent link="front_chassis_pitch_link"/>
         <child link="front_chassis"/>
-        <origin xyz="${scaled_chassis_length / 2}  0 0" rpy="0 0 0"/>
         <axis xyz="0 0 1"/>
-        <limit effort="200.0" lower="${-pi/3}" upper="${pi/3}" velocity="1.0"/>
+        <origin xyz="0 0 0" rpy="0 0 0"/>
+        <limit lower="-0.5" upper="0.5" effort="1000" velocity="1.0"/>
     </joint>
     <link name="front_chassis">
@@ -169,11 +193,11 @@
         </visual>
         <collision>
-            <origin xyz="${scaled_chassis_length / 2} 0 0" rpy="0 ${pi/2} 0"/>
-            <geometry>
-                <cylinder radius="${scaled_chassis_radius * 0.8}" length="${scaled_chassis_length * 0.8}"/>
+            <origin xyz="${scaled_chassis_length} 0 0" rpy="0 ${pi/2} 0"/>
+            <geometry>
+                <cylinder radius="${scaled_chassis_radius}" length="${scaled_chassis_length}"/>
             </geometry>
         </collision>
         <xacro:inertial_cylinder mass="${scaled_chassis_mass}" radius="${scaled_chassis_radius}" length="${scaled_chassis_length}">
-            <origin xyz="${scaled_chassis_length / 2} 0 0" rpy="0 ${pi/2} 0"/>
+            <origin xyz="${scaled_chassis_length} 0 0" rpy="0 ${pi/2} 0"/>
         </xacro:inertial_cylinder>
     </link>
@@ -182,9 +206,9 @@
     </gazebo>
     <!-- LEFT FRONT WHEEL LINK -->
-    <joint name="lf_wheel_joint" type="continuous">
+    <joint name="lf_wheel_joint" type="fixed">
         <parent link="front_chassis"/>
         <child link="lf_wheel"/>
         <origin xyz="${scaled_wheel_radius} ${scaled_chassis_radius} 0" rpy="-${pi/2} 0 0"/>
-        <axis xyz="0 0 1"/>
+        <!-- <axis xyz="0 0 1"/> -->
     </joint>
     <link name="lf_wheel">
@@ -208,11 +232,13 @@
     <gazebo reference="lf_wheel">
         <material>Gazebo/Red</material>
+        <mu1 value="0.001"/>
+        <mu2 value="0.001"/>
     </gazebo>
     <!-- RIGHT FRONT WHEEL LINK -->
-    <joint name="rf_wheel_joint" type="continuous">
+    <joint name="rf_wheel_joint" type="fixed">
         <parent link="front_chassis"/>
         <child link="rf_wheel"/>
         <origin xyz="${scaled_wheel_radius} -${scaled_chassis_radius} 0" rpy="${pi/2} 0 0"/>
-        <axis xyz="0 0 -1"/>
+        <!-- <axis xyz="0 0 -1"/> -->
     </joint>
     <link name="rf_wheel">
@@ -236,4 +262,6 @@
     <gazebo reference="rf_wheel">
         <material>Gazebo/Red</material>
+        <mu1 value="0.001"/>
+        <mu2 value="0.001"/>
     </gazebo>
     <!-- FRONT CASTER WHEEL LINK -->

File: description/robot_exe.xacro (robot description, xacro)
@@ -3,7 +3,6 @@
     <xacro:include filename="inertial_macros.xacro"/>
     <xacro:include filename="rgb_camera.xacro"/>
-    <xacro:include filename="robot_core_test.xacro"/>
+    <xacro:include filename="robot_core.xacro"/>
     <xacro:include filename="keyboard_control.xacro"/>
     <xacro:include filename="control.xacro"/>
-    <!-- <xacro:include filename="ros2_control.xacro"/> -->
 </robot>
