Commit message: 0403

File: description/control.xacro (robot description, xacro)
@@ -23,5 +23,5 @@
             <state_interface name="effort"/>
         </joint>
-        <joint name="front_chassis_roll_joint">
+        <joint name="chassis_roll_joint">
             <command_interface name="position">
                 <param name="min">-1</param>
@@ -32,5 +32,5 @@
             <state_interface name="effort"/>
         </joint>
-        <joint name="front_chassis_pitch_joint">
+        <joint name="chassis_pitch_joint">
             <command_interface name="position">
                 <param name="min">-1</param>
@@ -41,5 +41,5 @@
             <state_interface name="effort"/>
         </joint>
-        <joint name="front_chassis_yaw_joint">
+        <joint name="chassis_yaw_joint">
             <command_interface name="position">
                 <param name="min">-1</param>

File: description/depth_camera.xacro (robot description, xacro)
@@ -10,17 +10,25 @@
                 <horizontal_fov>1.089</horizontal_fov>
                 <image>
-                    <format>B8G8R8</format>
+                    <format>R8G8B8</format>
                     <width>640</width>
                     <height>480</height>
                 </image>
                 <clip>
-                    <near>0.05</near>
-                    <far>10.0</far>
+                    <near>0.02</near>
+                    <far>100.0</far>
                 </clip>
             </camera>
             <plugin name="camera_controller" filename="libgazebo_ros_camera.so">
                 <frame_name>camera_optical_link</frame_name>
-                <min_depth>0.1</min_depth>
+                <min_depth>0.02</min_depth>
                 <max_depth>100.0</max_depth>
+                <baseline>0.2</baseline>
+                <alwaysOn>true</alwaysOn>
+                <updateRate>1.0</updateRate>
+                <CxPrime>0</CxPrime>
+                <Cx>0</Cx>
+                <Cy>0</Cy>
+                <focalLength>0</focalLength>
+                <hackBaseline>0</hackBaseline>
             </plugin>
         </sensor>

File: description/inertial_macros.xacro (robot description, xacro)
@@ -1,4 +1,4 @@
 <?xml version="1.0"?>
-<robot xmlns:xacro="http://www.ros.org/wiki/xacro" >
+<robot xmlns:xacro="http://www.ros.org/wiki/xacro" name="colonoscopy">
     <!-- Specify some standard inertial calculations https://en.wikipedia.org/wiki/List_of_moments_of_inertia -->
     <!-- These make use of xacro's mathematical functionality -->

File: description/keyboard_control.xacro (robot description, xacro)
@@ -9,6 +9,6 @@
             <left_joint>lb_wheel_joint</left_joint>
             <right_joint>rb_wheel_joint</right_joint>
-            <wheel_separation>${2 * scaled_chassis_radius + scaled_wheel_length}</wheel_separation>
-            <wheel_diameter>${2 * scaled_wheel_radius}</wheel_diameter>
+            <wheel_separation>${2 * scaled_back_chassis_radius + scaled_back_wheel_length}</wheel_separation>
+            <wheel_diameter>${2 * scaled_back_wheel_radius}</wheel_diameter>
             <!-- Limits -->
             <max_wheel_torque>200</max_wheel_torque>

File: description/rgb_camera.xacro (robot description, xacro)
@@ -1,4 +1,4 @@
 <?xml version="1.0"?>
-<robot xmlns:xacro="http://www.ros.org/wiki/xacro">
+<robot xmlns:xacro="http://www.ros.org/wiki/xacro" name="colonoscopy">
     <gazebo reference="camera_link">
         <material>Gazebo/Red</material>

File: description/robot_core_test.xacro (robot description, xacro)
@@ -29,17 +29,20 @@
     <!-- Update All Parameters from a Single Parameter -->
     <xacro:property name="scale" value="50.0"/>
-    <xacro:property name="scaled_chassis_radius" value="${chassis_radius * scale}"/>
-    <xacro:property name="scaled_chassis_length" value="${chassis_length * scale}"/>
-    <xacro:property name="scaled_wheel_radius" value="${scaled_chassis_radius * 1.1}"/>
-    <xacro:property name="scaled_wheel_length" value="${wheel_length * scale}"/>
-    <xacro:property name="scaled_chassis_mass" value="${chassis_mass * scale}"/>
-    <xacro:property name="scaled_wheel_mass" value="${wheel_mass * scale}"/>
+    <xacro:property name="scaled_back_chassis_radius" value="${chassis_radius * scale}"/>
+    <xacro:property name="scaled_back_chassis_length" value="${chassis_length * scale}"/>
+    <xacro:property name="scaled_back_wheel_radius" value="${scaled_back_chassis_radius * 1.1}"/>
+    <xacro:property name="scaled_back_wheel_length" value="${wheel_length * scale}"/>
+    <xacro:property name="scaled_front_chassis_radius" value="${scaled_back_chassis_radius * 0.2}"/>
+    <xacro:property name="scaled_front_chassis_length" value="${scaled_back_chassis_length * 0.1}"/>
+    <xacro:property name="scaled_back_chassis_mass" value="${chassis_mass * scale}"/>
+    <xacro:property name="scaled_front_chassis_mass" value="${scaled_back_chassis_mass * 0.1}"/>
+    <xacro:property name="scaled_back_wheel_mass" value="${wheel_mass * scale}"/>
     <xacro:property name="scaled_caster_wheel_mass" value="${caster_wheel_mass * scale}"/>
-    <xacro:property name="scaled_camera_length" value="${scaled_chassis_radius / 5}"/>
+    <xacro:property name="scaled_camera_length" value="${scaled_back_chassis_radius / 5}"/>
     <!-- BACK CHASSIS LINK -->
     <joint name="back_chassis_joint" type="fixed">
         <parent link="base_link"/>
         <child link="back_chassis"/>
-        <origin xyz="${scaled_chassis_length / 2} 0 ${scaled_wheel_radius}" rpy="0 0 0"/>
+        <origin xyz="${scaled_back_chassis_length / 2} 0 ${scaled_back_wheel_radius}" rpy="0 0 0"/>
     </joint>
     <link name="back_chassis">
@@ -47,5 +50,5 @@
             <origin xyz="0 0 0" rpy="0 ${pi/2} 0"/>
             <geometry>
-                <cylinder radius="${scaled_chassis_radius}" length="${scaled_chassis_length}"/>
+                <cylinder radius="${scaled_back_chassis_radius}" length="${scaled_back_chassis_length}"/>
             </geometry>
             <material name="white"/>
@@ -54,8 +57,8 @@
             <origin xyz="0 0 0" rpy="0 ${pi/2} 0"/>
             <geometry>
-                <cylinder radius="${scaled_chassis_radius * 0.8}" length="${scaled_chassis_length * 0.8}"/>
-            </geometry>
-        </collision>
-        <xacro:inertial_cylinder mass="${scaled_chassis_mass}" radius="${scaled_chassis_radius}" length="${scaled_chassis_length}">
+                <cylinder radius="${scaled_back_chassis_radius * 0.8}" length="${scaled_back_chassis_length * 0.8}"/>
+            </geometry>
+        </collision>
+        <xacro:inertial_cylinder mass="${scaled_back_chassis_mass}" radius="${scaled_back_chassis_radius}" length="${scaled_back_chassis_length}">
             <origin xyz="0 0 0" rpy="0 ${pi/2} 0"/>
         </xacro:inertial_cylinder>
@@ -68,23 +71,23 @@
         <parent link="base_link"/>
         <child link="lb_wheel"/>
-        <origin xyz="${scaled_wheel_radius} ${scaled_chassis_radius} ${scaled_wheel_radius}" rpy="-${pi/2} 0 0" />
+        <origin xyz="${scaled_back_wheel_radius} ${scaled_back_chassis_radius} ${scaled_back_wheel_radius}" rpy="-${pi/2} 0 0" />
         <axis xyz="0 0 1"/>
     </joint>
     <link name="lb_wheel">
         <visual>
-            <origin xyz="0 0 ${scaled_wheel_length / 2}" rpy="0 0 0"/>
-            <geometry>
-                <cylinder radius="${scaled_wheel_radius}" length="${scaled_wheel_length}"/>
+            <origin xyz="0 0 ${scaled_back_wheel_length / 2}" rpy="0 0 0"/>
+            <geometry>
+                <cylinder radius="${scaled_back_wheel_radius}" length="${scaled_back_wheel_length}"/>
             </geometry>
             <material name="blue"/>
         </visual>
         <collision>
-            <origin xyz="0 0 ${scaled_wheel_length / 2}" rpy="0 0 0"/>
-            <geometry>
-                <cylinder radius="${scaled_wheel_radius}" length="${scaled_wheel_length}"/>
-            </geometry>
-        </collision>
-        <xacro:inertial_cylinder mass="${scaled_wheel_mass}" radius="${scaled_wheel_radius}" length="${scaled_wheel_length}">
-            <origin xyz="0 0 ${scaled_wheel_length / 2}" rpy="0 0 0"/>
+            <origin xyz="0 0 ${scaled_back_wheel_length / 2}" rpy="0 0 0"/>
+            <geometry>
+                <cylinder radius="${scaled_back_wheel_radius}" length="${scaled_back_wheel_length}"/>
+            </geometry>
+        </collision>
+        <xacro:inertial_cylinder mass="${scaled_back_wheel_mass}" radius="${scaled_back_wheel_radius}" length="${scaled_back_wheel_length}">
+            <origin xyz="0 0 ${scaled_back_wheel_length / 2}" rpy="0 0 0"/>
         </xacro:inertial_cylinder>
     </link>
@@ -96,23 +99,23 @@
         <parent link="base_link"/>
         <child link="rb_wheel"/>
-        <origin xyz="${scaled_wheel_radius} -${scaled_chassis_radius} ${scaled_wheel_radius}" rpy="${pi/2} 0 0" />
+        <origin xyz="${scaled_back_wheel_radius} -${scaled_back_chassis_radius} ${scaled_back_wheel_radius}" rpy="${pi/2} 0 0" />
         <axis xyz="0 0 -1"/>
     </joint>
     <link name="rb_wheel">
         <visual>
-            <origin xyz="0 0 ${scaled_wheel_length / 2}" rpy="0 0 0"/>
-            <geometry>
-                <cylinder radius="${scaled_wheel_radius}" length="${scaled_wheel_length}"/>
+            <origin xyz="0 0 ${scaled_back_wheel_length / 2}" rpy="0 0 0"/>
+            <geometry>
+                <cylinder radius="${scaled_back_wheel_radius}" length="${scaled_back_wheel_length}"/>
             </geometry>
             <material name="blue"/>
         </visual>
         <collision>
-            <origin xyz="0 0 ${scaled_wheel_length / 2}" rpy="0 0 0"/>
-            <geometry>
-                <cylinder radius="${scaled_wheel_radius}" length="${scaled_wheel_length}"/>
-            </geometry>
-        </collision>
-        <xacro:inertial_cylinder mass="${scaled_wheel_mass}" radius="${scaled_wheel_radius}" length="${scaled_wheel_length}">
-            <origin xyz="0 0 ${scaled_wheel_length / 2}" rpy="0 0 0"/>
+            <origin xyz="0 0 ${scaled_back_wheel_length / 2}" rpy="0 0 0"/>
+            <geometry>
+                <cylinder radius="${scaled_back_wheel_radius}" length="${scaled_back_wheel_length}"/>
+            </geometry>
+        </collision>
+        <xacro:inertial_cylinder mass="${scaled_back_wheel_mass}" radius="${scaled_back_wheel_radius}" length="${scaled_back_wheel_length}">
+            <origin xyz="0 0 ${scaled_back_wheel_length / 2}" rpy="0 0 0"/>
         </xacro:inertial_cylinder>
     </link>
@@ -124,10 +127,10 @@
         <parent link="back_chassis"/>
         <child link="b_caster_wheel"/>
-        <origin xyz="${scaled_chassis_length / 4} 0 -${scaled_wheel_radius / 2}" rpy="0 0 0"/>
+        <origin xyz="${scaled_back_chassis_length / 4} 0 -${scaled_back_wheel_radius / 2}" rpy="0 0 0"/>
     </joint>
     <link name="b_caster_wheel">
         <visual>
             <geometry>
-                <sphere radius="${scaled_wheel_radius / 2}"/>
+                <sphere radius="${scaled_back_wheel_radius / 2}"/>
             </geometry>
             <material name="black"/>
@@ -135,8 +138,8 @@
         <collision>
             <geometry>
-                <sphere radius="${scaled_wheel_radius / 2}"/>
-            </geometry>
-        </collision>
-        <xacro:inertial_sphere mass="${scaled_caster_wheel_mass}" radius="${scaled_wheel_radius / 2}">
+                <sphere radius="${scaled_back_wheel_radius / 2}"/>
+            </geometry>
+        </collision>
+        <xacro:inertial_sphere mass="${scaled_caster_wheel_mass}" radius="${scaled_back_wheel_radius / 2}">
             <origin xyz="0 0 0" rpy="0 0 0"/>
         </xacro:inertial_sphere>
@@ -151,8 +154,8 @@
         <parent link="back_chassis"/>
         <child link="chassis_roll_link"/>
-        <origin xyz="${scaled_chassis_length / 2}  0 0" rpy="0 0 0"/>
+        <origin xyz="${scaled_back_chassis_length / 2}  0 0" rpy="0 0 0"/>
         <axis xyz="-1 0 0"/>
-        <limit lower="-0.5" upper="0.5" effort="1000.0" velocity="1.0"/>
-        <dynamics damping="1.0" friction="0.1"/>
+        <limit lower="-${pi / 4}" upper="${pi / 4}" effort="1000.0" velocity="1.0"/>
+        <!-- <dynamics damping="1.0" friction="0.1"/> -->
     </joint>
     <link name="chassis_roll_link">
@@ -168,5 +171,5 @@
         <axis xyz="0 1 0"/>
         <origin xyz="0 0 0" rpy="0 0 0"/>
-        <limit lower="-0.5" upper="0.5" effort="1000" velocity="1.0"/>
+        <limit lower="-${pi / 4}" upper="${pi / 4}" effort="1000.0" velocity="1.0"/>
     </joint>
     <link name="chassis_pitch_link">
@@ -182,22 +185,22 @@
         <axis xyz="0 0 1"/>
         <origin xyz="0 0 0" rpy="0 0 0"/>
-        <limit lower="-0.5" upper="0.5" effort="1000" velocity="1.0"/>
+        <limit lower="-${pi / 4}" upper="${pi / 4}" effort="1000.0" velocity="1.0"/>
     </joint>
     <link name="front_chassis">
         <visual>
-            <origin xyz="${scaled_chassis_length / 2} 0 0" rpy="0 ${pi/2} 0"/>
-            <geometry>
-                <cylinder radius="${scaled_chassis_radius}" length="${scaled_chassis_length}"/>
+            <origin xyz="${scaled_front_chassis_length / 2} 0 0" rpy="0 ${pi/2} 0"/>
+            <geometry>
+                <cylinder radius="${scaled_front_chassis_radius}" length="${scaled_front_chassis_length}"/>
             </geometry>
             <material name="white"/>
         </visual>
         <collision>
-            <origin xyz="${scaled_chassis_length} 0 0" rpy="0 ${pi/2} 0"/>
-            <geometry>
-                <cylinder radius="${scaled_chassis_radius}" length="${scaled_chassis_length}"/>
-            </geometry>
-        </collision>
-        <xacro:inertial_cylinder mass="${scaled_chassis_mass}" radius="${scaled_chassis_radius}" length="${scaled_chassis_length}">
-            <origin xyz="${scaled_chassis_length} 0 0" rpy="0 ${pi/2} 0"/>
+            <origin xyz="${scaled_front_chassis_length / 2} 0 0" rpy="0 ${pi/2} 0"/>
+            <geometry>
+                <cylinder radius="${scaled_front_chassis_radius}" length="${scaled_front_chassis_length / 10}"/>
+            </geometry>
+        </collision>
+        <xacro:inertial_cylinder mass="${scaled_front_chassis_mass}" radius="${scaled_front_chassis_radius / 5}" length="${scaled_back_chassis_length}">
+            <origin xyz="${scaled_front_chassis_length / 2} 0 0" rpy="0 ${pi/2} 0"/>
         </xacro:inertial_cylinder>
     </link>
@@ -206,26 +209,25 @@
     </gazebo>
     <!-- LEFT FRONT WHEEL LINK -->
-    <joint name="lf_wheel_joint" type="fixed">
+    <!-- <joint name="lf_wheel_joint" type="fixed">
         <parent link="front_chassis"/>
         <child link="lf_wheel"/>
-        <origin xyz="${scaled_wheel_radius} ${scaled_chassis_radius} 0" rpy="-${pi/2} 0 0"/>
-        <!-- <axis xyz="0 0 1"/> -->
+        <origin xyz="${scaled_back_wheel_radius} ${scaled_back_chassis_radius} 0" rpy="-${pi/2} 0 0"/>
     </joint>
     <link name="lf_wheel">
         <visual>
-            <origin xyz="0 0 ${scaled_wheel_length / 2}" rpy="0 0 0"/>
-            <geometry>
-                <cylinder radius="${scaled_wheel_radius}" length="${scaled_wheel_length}"/>
+            <origin xyz="0 0 ${scaled_back_wheel_length / 2}" rpy="0 0 0"/>
+            <geometry>
+                <cylinder radius="${scaled_back_wheel_radius}" length="${scaled_back_wheel_length}"/>
             </geometry>
             <material name="red"/>
         </visual>
         <collision>
-            <origin xyz="0 0 ${scaled_wheel_length / 2}" rpy="0 0 0"/>
-            <geometry>
-                <cylinder radius="${scaled_wheel_radius}" length="${scaled_wheel_length}"/>
-            </geometry>
-        </collision>
-        <xacro:inertial_cylinder mass="${scaled_wheel_mass}" radius="${scaled_wheel_radius}" length="${scaled_wheel_length}">
-            <origin xyz="0 0 ${scaled_wheel_length / 2}" rpy="0 0 0"/>
+            <origin xyz="0 0 ${scaled_back_wheel_length / 2}" rpy="0 0 0"/>
+            <geometry>
+                <cylinder radius="${scaled_back_wheel_radius}" length="${scaled_back_wheel_length}"/>
+            </geometry>
+        </collision>
+        <xacro:inertial_cylinder mass="${scaled_back_wheel_mass}" radius="${scaled_back_wheel_radius}" length="${scaled_back_wheel_length}">
+            <origin xyz="0 0 ${scaled_back_wheel_length / 2}" rpy="0 0 0"/>
         </xacro:inertial_cylinder>
     </link>
@@ -234,28 +236,27 @@
         <mu1 value="0.001"/>
         <mu2 value="0.001"/>
-    </gazebo>
+    </gazebo> -->
     <!-- RIGHT FRONT WHEEL LINK -->
-    <joint name="rf_wheel_joint" type="fixed">
+    <!-- <joint name="rf_wheel_joint" type="fixed">
         <parent link="front_chassis"/>
         <child link="rf_wheel"/>
-        <origin xyz="${scaled_wheel_radius} -${scaled_chassis_radius} 0" rpy="${pi/2} 0 0"/>
-        <!-- <axis xyz="0 0 -1"/> -->
+        <origin xyz="${scaled_back_wheel_radius} -${scaled_back_chassis_radius} 0" rpy="${pi/2} 0 0"/>
     </joint>
     <link name="rf_wheel">
         <visual>
-            <origin xyz="0 0 ${scaled_wheel_length / 2}" rpy="0 0 0"/>
-            <geometry>
-                <cylinder radius="${scaled_wheel_radius}" length="${scaled_wheel_length}"/>
+            <origin xyz="0 0 ${scaled_back_wheel_length / 2}" rpy="0 0 0"/>
+            <geometry>
+                <cylinder radius="${scaled_back_wheel_radius}" length="${scaled_back_wheel_length}"/>
             </geometry>
             <material name="red"/>
         </visual>
         <collision>
-            <origin xyz="0 0 ${scaled_wheel_length / 2}" rpy="0 0 0"/>
-            <geometry>
-                <cylinder radius="${scaled_wheel_radius}" length="${scaled_wheel_length}"/>
-            </geometry>
-        </collision>
-        <xacro:inertial_cylinder mass="${scaled_wheel_mass}" radius="${scaled_wheel_radius}" length="${scaled_wheel_length}">
-            <origin xyz="0 0 ${scaled_wheel_length / 2}" rpy="0 0 0"/>
+            <origin xyz="0 0 ${scaled_back_wheel_length / 2}" rpy="0 0 0"/>
+            <geometry>
+                <cylinder radius="${scaled_back_wheel_radius}" length="${scaled_back_wheel_length}"/>
+            </geometry>
+        </collision>
+        <xacro:inertial_cylinder mass="${scaled_back_wheel_mass}" radius="${scaled_back_wheel_radius}" length="${scaled_back_wheel_length}">
+            <origin xyz="0 0 ${scaled_back_wheel_length / 2}" rpy="0 0 0"/>
         </xacro:inertial_cylinder>
     </link>
@@ -264,15 +265,15 @@
         <mu1 value="0.001"/>
         <mu2 value="0.001"/>
-    </gazebo>
+    </gazebo> -->
     <!-- FRONT CASTER WHEEL LINK -->
-    <joint name="f_caster_wheel_joint" type="fixed">
+    <!-- <joint name="f_caster_wheel_joint" type="fixed">
         <parent link="front_chassis"/>
         <child link="f_caster_wheel"/>
-        <origin xyz="${scaled_chassis_length * 0.75} 0 -${scaled_wheel_radius / 2}" rpy="0 0 0"/>
+        <origin xyz="${scaled_back_chassis_length * 0.75} 0 -${scaled_back_wheel_radius / 2}" rpy="0 0 0"/>
     </joint>
     <link name="f_caster_wheel">
         <visual>
             <geometry>
-                <sphere radius="${scaled_wheel_radius / 2}"/>
+                <sphere radius="${scaled_back_wheel_radius / 2}"/>
             </geometry>
             <material name="black"/>
@@ -280,8 +281,8 @@
         <collision>
             <geometry>
-                <sphere radius="${scaled_wheel_radius / 2}"/>
-            </geometry>
-        </collision>
-        <xacro:inertial_sphere mass="${scaled_caster_wheel_mass}" radius="${scaled_wheel_radius / 2}">
+                <sphere radius="${scaled_back_wheel_radius / 2}"/>
+            </geometry>
+        </collision>
+        <xacro:inertial_sphere mass="${scaled_caster_wheel_mass}" radius="${scaled_back_wheel_radius / 2}">
             <origin xyz="0 0 0" rpy="0 0 0"/>
         </xacro:inertial_sphere>
@@ -291,10 +292,10 @@
         <mu1 value="0.001"/>
         <mu2 value="0.001"/>
-    </gazebo>
+    </gazebo> -->
     <!-- CAMERA -->
     <joint name="camera_joint" type="fixed">
         <parent link="front_chassis"/>
         <child link="camera_link"/>
-        <origin xyz="${scaled_chassis_length} 0 0" rpy="0 0 0"/>
+        <origin xyz="${scaled_front_chassis_length} 0 0" rpy="0 0 0"/>
     </joint>
     <link name="camera_link">

File: description/robot_exe.xacro (robot description, xacro)
@@ -2,6 +2,6 @@
 <robot xmlns:xacro="http://www.ros.org/wiki/xacro" name="colonoscopy">
     <xacro:include filename="inertial_macros.xacro"/>
-    <xacro:include filename="rgb_camera.xacro"/>
-    <xacro:include filename="robot_core.xacro"/>
+    <xacro:include filename="depth_camera.xacro"/>
+    <xacro:include filename="robot_core_test.xacro"/>
     <xacro:include filename="keyboard_control.xacro"/>
     <xacro:include filename="control.xacro"/>
