Commit message: 0404

File: description/depth_camera.xacro (robot description, xacro)
@@ -23,12 +23,4 @@
                 <min_depth>0.02</min_depth>
                 <max_depth>100.0</max_depth>
-                <baseline>0.2</baseline>
-                <alwaysOn>true</alwaysOn>
-                <updateRate>1.0</updateRate>
-                <CxPrime>0</CxPrime>
-                <Cx>0</Cx>
-                <Cy>0</Cy>
-                <focalLength>0</focalLength>
-                <hackBaseline>0</hackBaseline>
             </plugin>
         </sensor>

File: description/keyboard_control.xacro (robot description, xacro)
@@ -15,4 +15,5 @@
             <max_wheel_acceleration>10.0</max_wheel_acceleration>
             <!-- Output -->
+            <odometry_topic>odom</odometry_topic>
             <odometry_frame>odom</odometry_frame>
             <robot_base_frame>base_link</robot_base_frame>

File: description/robot_core.xacro (robot description, xacro)
@@ -21,25 +21,28 @@
     <!-- DEFINE PARAMETERS -->
     <xacro:property name="chassis_radius" value="0.0065"/>
-    <xacro:property name="chassis_length" value="0.03"/>
-    <xacro:property name="wheel_radius" value="0.008"/>
-    <xacro:property name="wheel_length" value="0.001"/>
+    <xacro:property name="chassis_length" value="${chassis_radius * 5}"/>
+    <xacro:property name="wheel_radius" value="${chassis_radius * 1.2}"/>
+    <xacro:property name="wheel_length" value="${chassis_length * 0.1}"/>
     <xacro:property name="chassis_mass" value="1.0"/>
     <xacro:property name="wheel_mass" value="0.005"/>
-    <xacro:property name="caster_wheel_mass" value="0.005"/>
+    <xacro:property name="caster_wheel_mass" value="0.01"/>
     <!-- Update All Parameters from a Single Parameter -->
     <xacro:property name="scale" value="50.0"/>
-    <xacro:property name="scaled_chassis_radius" value="${chassis_radius * scale}"/>
-    <xacro:property name="scaled_chassis_length" value="${chassis_length * scale}"/>
-    <xacro:property name="scaled_wheel_radius" value="${scaled_chassis_radius * 1.1}"/>
-    <xacro:property name="scaled_wheel_length" value="${wheel_length * scale}"/>
+    <xacro:property name="scaled_back_chassis_radius" value="${chassis_radius * scale}"/>
+    <xacro:property name="scaled_back_chassis_length" value="${chassis_length * scale}"/>
+    <xacro:property name="scaled_front_chassis_radius" value="${scaled_back_chassis_radius * 0.5}"/>
+    <xacro:property name="scaled_front_chassis_length" value="${scaled_back_chassis_length * 0.5}"/>
+    <xacro:property name="scaled_back_wheel_radius" value="${wheel_radius * scale}"/>
+    <xacro:property name="scaled_back_wheel_length" value="${wheel_length * scale}"/>
     <xacro:property name="scaled_chassis_mass" value="${chassis_mass * scale}"/>
+    <xacro:property name="scaled_front_chassis_mass" value="${scaled_chassis_mass * 0.2}"/>
     <xacro:property name="scaled_wheel_mass" value="${wheel_mass * scale}"/>
     <xacro:property name="scaled_caster_wheel_mass" value="${caster_wheel_mass * scale}"/>
-    <xacro:property name="scaled_camera_length" value="${scaled_chassis_radius / 5}"/>
+    <xacro:property name="scaled_camera_length" value="${scaled_back_chassis_radius * 0.2}"/>
     <!-- BACK CHASSIS LINK -->
     <joint name="back_chassis_joint" type="fixed">
         <parent link="base_link"/>
         <child link="back_chassis"/>
-        <origin xyz="${scaled_chassis_length / 2} 0 ${scaled_wheel_radius}" rpy="0 0 0"/>
+        <origin xyz="${scaled_back_chassis_length / 2} 0 ${scaled_back_wheel_radius}" rpy="0 0 0"/>
     </joint>
     <link name="back_chassis">
@@ -47,44 +50,43 @@
             <origin xyz="0 0 0" rpy="0 ${pi/2} 0"/>
             <geometry>
-                <cylinder radius="${scaled_chassis_radius}" length="${scaled_chassis_length}"/>
-            </geometry>
-            <material name="white"/>
+                <cylinder radius="${scaled_back_chassis_radius}" length="${scaled_back_chassis_length}"/>
+            </geometry>
+            <material name="black"/>
         </visual>
         <collision>
             <origin xyz="0 0 0" rpy="0 ${pi/2} 0"/>
             <geometry>
-                <cylinder radius="${scaled_chassis_radius * 0.8}" length="${scaled_chassis_length * 0.8}"/>
-            </geometry>
-        </collision>
-        <xacro:inertial_cylinder mass="${scaled_chassis_mass}" radius="${scaled_chassis_radius}" length="${scaled_chassis_length}">
+                <cylinder radius="${scaled_back_chassis_radius}" length="${scaled_back_chassis_length - scaled_front_chassis_radius}"/>
+            </geometry>
+        </collision>
+        <xacro:inertial_cylinder mass="${scaled_chassis_mass}" radius="${scaled_back_chassis_radius}" length="${scaled_back_chassis_length}">
             <origin xyz="0 0 0" rpy="0 ${pi/2} 0"/>
         </xacro:inertial_cylinder>
     </link>
     <gazebo reference="back_chassis">
-        <material>Gazebo/White</material>
-    </gazebo>
-    <!-- LEFT BACK WHEEL LINK -->
+        <material>Gazebo/Black</material>
+    </gazebo>
     <joint name="lb_wheel_joint" type="continuous">
-        <parent link="base_link"/>
+        <parent link="back_chassis"/>
         <child link="lb_wheel"/>
-        <origin xyz="${scaled_wheel_radius} ${scaled_chassis_radius} ${scaled_wheel_radius}" rpy="-${pi/2} 0 0" />
+        <origin xyz="${scaled_back_wheel_radius - scaled_back_chassis_length / 2} ${scaled_back_chassis_radius} 0" rpy="-${pi/2} 0 0" />
         <axis xyz="0 0 1"/>
     </joint>
     <link name="lb_wheel">
         <visual>
-            <origin xyz="0 0 ${scaled_wheel_length / 2}" rpy="0 0 0"/>
-            <geometry>
-                <cylinder radius="${scaled_wheel_radius}" length="${scaled_wheel_length}"/>
+            <origin xyz="0 0 ${scaled_back_wheel_length / 2}" rpy="0 0 0"/>
+            <geometry>
+                <cylinder radius="${scaled_back_wheel_radius}" length="${scaled_back_wheel_length}"/>
             </geometry>
             <material name="blue"/>
         </visual>
         <collision>
-            <origin xyz="0 0 ${scaled_wheel_length / 2}" rpy="0 0 0"/>
-            <geometry>
-                <cylinder radius="${scaled_wheel_radius}" length="${scaled_wheel_length}"/>
-            </geometry>
-        </collision>
-        <xacro:inertial_cylinder mass="${scaled_wheel_mass}" radius="${scaled_wheel_radius}" length="${scaled_wheel_length}">
-            <origin xyz="0 0 ${scaled_wheel_length / 2}" rpy="0 0 0"/>
+            <origin xyz="0 0 ${scaled_back_wheel_length / 2}" rpy="0 0 0"/>
+            <geometry>
+                <cylinder radius="${scaled_back_wheel_radius}" length="${scaled_back_wheel_length}"/>
+            </geometry>
+        </collision>
+        <xacro:inertial_cylinder mass="${scaled_wheel_mass}" radius="${scaled_back_wheel_radius}" length="${scaled_back_wheel_length}">
+            <origin xyz="0 0 ${scaled_back_wheel_length / 2}" rpy="0 0 0"/>
         </xacro:inertial_cylinder>
     </link>
@@ -92,27 +94,26 @@
         <material>Gazebo/Blue</material>
     </gazebo>
-    <!-- RIGHT BACK WHEEL LINK -->
     <joint name="rb_wheel_joint" type="continuous">
-        <parent link="base_link"/>
+        <parent link="back_chassis"/>
         <child link="rb_wheel"/>
-        <origin xyz="${scaled_wheel_radius} -${scaled_chassis_radius} ${scaled_wheel_radius}" rpy="${pi/2} 0 0" />
+        <origin xyz="${scaled_back_wheel_radius - scaled_back_chassis_length / 2} -${scaled_back_chassis_radius} 0" rpy="${pi/2} 0 0" />
         <axis xyz="0 0 -1"/>
     </joint>
     <link name="rb_wheel">
         <visual>
-            <origin xyz="0 0 ${scaled_wheel_length / 2}" rpy="0 0 0"/>
-            <geometry>
-                <cylinder radius="${scaled_wheel_radius}" length="${scaled_wheel_length}"/>
+            <origin xyz="0 0 ${scaled_back_wheel_length / 2}" rpy="0 0 0"/>
+            <geometry>
+                <cylinder radius="${scaled_back_wheel_radius}" length="${scaled_back_wheel_length}"/>
             </geometry>
             <material name="blue"/>
         </visual>
         <collision>
-            <origin xyz="0 0 ${scaled_wheel_length / 2}" rpy="0 0 0"/>
-            <geometry>
-                <cylinder radius="${scaled_wheel_radius}" length="${scaled_wheel_length}"/>
-            </geometry>
-        </collision>
-        <xacro:inertial_cylinder mass="${scaled_wheel_mass}" radius="${scaled_wheel_radius}" length="${scaled_wheel_length}">
-            <origin xyz="0 0 ${scaled_wheel_length / 2}" rpy="0 0 0"/>
+            <origin xyz="0 0 ${scaled_back_wheel_length / 2}" rpy="0 0 0"/>
+            <geometry>
+                <cylinder radius="${scaled_back_wheel_radius}" length="${scaled_back_wheel_length}"/>
+            </geometry>
+        </collision>
+        <xacro:inertial_cylinder mass="${scaled_wheel_mass}" radius="${scaled_back_wheel_radius}" length="${scaled_back_wheel_length}">
+            <origin xyz="0 0 ${scaled_back_wheel_length / 2}" rpy="0 0 0"/>
         </xacro:inertial_cylinder>
     </link>
@@ -120,39 +121,68 @@
         <material>Gazebo/Blue</material>
     </gazebo>
-    <!-- BACK CASTER WHEEL LINK -->
-    <joint name="b_caster_wheel_joint" type="fixed">
-        <parent link="back_chassis"/>
-        <child link="b_caster_wheel"/>
-        <origin xyz="${scaled_chassis_length / 4} 0 -${scaled_wheel_radius / 2}" rpy="0 0 0"/>
-    </joint>
-    <link name="b_caster_wheel">
-        <visual>
-            <geometry>
-                <sphere radius="${scaled_wheel_radius / 2}"/>
-            </geometry>
-            <material name="black"/>
-        </visual>
-        <collision>
-            <geometry>
-                <sphere radius="${scaled_wheel_radius / 2}"/>
-            </geometry>
-        </collision>
-        <xacro:inertial_sphere mass="${scaled_caster_wheel_mass}" radius="${scaled_wheel_radius / 2}">
-            <origin xyz="0 0 0" rpy="0 0 0"/>
-        </xacro:inertial_sphere>
-    </link>
-    <gazebo reference="b_caster_wheel">
-        <material>Gazebo/Black</material>
-        <mu1 value="0.001"/>
-        <mu2 value="0.001"/>
-    </gazebo>
-    <!-- CHASSIS BETWEEN JOINT -->
+    <joint name="lb2_wheel_joint" type="continuous">
+        <parent link="back_chassis"/>
+        <child link="lb2_wheel"/>
+        <origin xyz="${scaled_back_chassis_length / 2 - scaled_back_wheel_radius} ${scaled_back_chassis_radius} 0" rpy="-${pi/2} 0 0"/>
+        <axis xyz="0 0 1"/>
+    </joint>
+    <link name="lb2_wheel">
+        <visual>
+            <origin xyz="0 0 ${scaled_back_wheel_length / 2}" rpy="0 0 0"/>
+            <geometry>
+                <cylinder radius="${scaled_back_wheel_radius}" length="${scaled_back_wheel_length}"/>
+            </geometry>
+            <material name="blue"/>
+        </visual>
+        <collision>
+            <origin xyz="0 0 ${scaled_back_wheel_length / 2}" rpy="0 0 0"/>
+            <geometry>
+                <cylinder radius="${scaled_back_wheel_radius}" length="${scaled_back_wheel_length}"/>
+            </geometry>
+        </collision>
+        <xacro:inertial_cylinder mass="${scaled_wheel_mass}" radius="${scaled_back_wheel_radius}" length="${scaled_back_wheel_length}">
+            <origin xyz="0 0 ${scaled_back_wheel_length / 2}" rpy="0 0 0"/>
+        </xacro:inertial_cylinder>
+    </link>
+    <gazebo reference="lb2_wheel">
+        <material>Gazebo/Blue</material>
+        <mu1 value="0.001"/>
+        <mu2 value="0.001"/>
+    </gazebo>
+    <joint name="rb2_wheel_joint" type="continuous">
+        <parent link="back_chassis"/>
+        <child link="rb2_wheel"/>
+        <origin xyz="${scaled_back_chassis_length / 2 - scaled_back_wheel_radius} -${scaled_back_chassis_radius} 0" rpy="${pi/2} 0 0"/>
+        <axis xyz="0 0 -1"/>
+    </joint>
+    <link name="rb2_wheel">
+        <visual>
+            <origin xyz="0 0 ${scaled_back_wheel_length / 2}" rpy="0 0 0"/>
+            <geometry>
+                <cylinder radius="${scaled_back_wheel_radius}" length="${scaled_back_wheel_length}"/>
+            </geometry>
+            <material name="blue"/>
+        </visual>
+        <collision>
+            <origin xyz="0 0 ${scaled_back_wheel_length / 2}" rpy="0 0 0"/>
+            <geometry>
+                <cylinder radius="${scaled_back_wheel_radius}" length="${scaled_back_wheel_length}"/>
+            </geometry>
+        </collision>
+        <xacro:inertial_cylinder mass="${scaled_wheel_mass}" radius="${scaled_back_wheel_radius}" length="${scaled_back_wheel_length}">
+            <origin xyz="0 0 ${scaled_back_wheel_length / 2}" rpy="0 0 0"/>
+        </xacro:inertial_cylinder>
+    </link>
+    <gazebo reference="rb2_wheel">
+        <material>Gazebo/Blue</material>
+        <mu1 value="0.001"/>
+        <mu2 value="0.001"/>
+    </gazebo>
     <joint name="chassis_roll_joint" type="revolute">
         <parent link="back_chassis"/>
         <child link="chassis_roll_link"/>
-        <origin xyz="${scaled_chassis_length / 2}  0 0" rpy="0 0 0"/>
+        <origin xyz="${scaled_back_chassis_length / 2}  0 0" rpy="0 0 0"/>
         <axis xyz="-1 0 0"/>
-        <limit lower="-0.5" upper="0.5" effort="1000.0" velocity="1.0"/>
-        <dynamics damping="1.0" friction="0.1"/>
+        <limit lower="-0.5" upper="0.5" effort="1000" velocity="1.0"/>
     </joint>
     <link name="chassis_roll_link">
@@ -162,5 +192,4 @@
         </inertial>
     </link>
-    <!-- Pitch Joint -->
     <joint name="chassis_pitch_joint" type="revolute">
         <parent link="chassis_roll_link"/>
@@ -176,5 +205,4 @@
         </inertial>
     </link>
-    <!-- Yaw Joint -->
     <joint name="chassis_yaw_joint" type="revolute">
         <parent link="chassis_pitch_link"/>
@@ -186,18 +214,18 @@
     <link name="front_chassis">
         <visual>
-            <origin xyz="${scaled_chassis_length / 2} 0 0" rpy="0 ${pi/2} 0"/>
-            <geometry>
-                <cylinder radius="${scaled_chassis_radius}" length="${scaled_chassis_length}"/>
+            <origin xyz="${scaled_front_chassis_length / 2} 0 0" rpy="0 ${pi/2} 0"/>
+            <geometry>
+                <cylinder radius="${scaled_front_chassis_radius}" length="${scaled_front_chassis_length}"/>
             </geometry>
             <material name="white"/>
         </visual>
         <collision>
-            <origin xyz="${scaled_chassis_length} 0 0" rpy="0 ${pi/2} 0"/>
-            <geometry>
-                <cylinder radius="${scaled_chassis_radius}" length="${scaled_chassis_length}"/>
-            </geometry>
-        </collision>
-        <xacro:inertial_cylinder mass="${scaled_chassis_mass}" radius="${scaled_chassis_radius}" length="${scaled_chassis_length}">
-            <origin xyz="${scaled_chassis_length} 0 0" rpy="0 ${pi/2} 0"/>
+            <origin xyz="${scaled_front_chassis_length / 2} 0 0" rpy="0 ${pi/2} 0"/>
+            <geometry>
+                <cylinder radius="${scaled_front_chassis_radius}" length="${scaled_front_chassis_length - scaled_front_chassis_radius}"/>
+            </geometry>
+        </collision>
+        <xacro:inertial_cylinder mass="${scaled_front_chassis_mass}" radius="${scaled_front_chassis_radius}" length="${scaled_front_chassis_length}">
+            <origin xyz="${scaled_front_chassis_length / 2} 0 0" rpy="0 ${pi/2} 0"/>
         </xacro:inertial_cylinder>
     </link>
@@ -205,27 +233,25 @@
         <material>Gazebo/White</material>
     </gazebo>
-    <!-- LEFT FRONT WHEEL LINK -->
-    <joint name="lf_wheel_joint" type="fixed">
+    <!-- <joint name="lf_wheel_joint" type="fixed">
         <parent link="front_chassis"/>
         <child link="lf_wheel"/>
-        <origin xyz="${scaled_wheel_radius} ${scaled_chassis_radius} 0" rpy="-${pi/2} 0 0"/>
-        <!-- <axis xyz="0 0 1"/> -->
+        <origin xyz="${scaled_back_wheel_radius} ${scaled_back_chassis_radius} 0" rpy="-${pi/2} 0 0"/>
     </joint>
     <link name="lf_wheel">
         <visual>
-            <origin xyz="0 0 ${scaled_wheel_length / 2}" rpy="0 0 0"/>
-            <geometry>
-                <cylinder radius="${scaled_wheel_radius}" length="${scaled_wheel_length}"/>
+            <origin xyz="0 0 ${scaled_back_wheel_length / 2}" rpy="0 0 0"/>
+            <geometry>
+                <cylinder radius="${scaled_back_wheel_radius}" length="${scaled_back_wheel_length}"/>
             </geometry>
             <material name="red"/>
         </visual>
         <collision>
-            <origin xyz="0 0 ${scaled_wheel_length / 2}" rpy="0 0 0"/>
-            <geometry>
-                <cylinder radius="${scaled_wheel_radius}" length="${scaled_wheel_length}"/>
-            </geometry>
-        </collision>
-        <xacro:inertial_cylinder mass="${scaled_wheel_mass}" radius="${scaled_wheel_radius}" length="${scaled_wheel_length}">
-            <origin xyz="0 0 ${scaled_wheel_length / 2}" rpy="0 0 0"/>
+            <origin xyz="0 0 ${scaled_back_wheel_length / 2}" rpy="0 0 0"/>
+            <geometry>
+                <cylinder radius="${scaled_back_wheel_radius}" length="${scaled_back_wheel_length}"/>
+            </geometry>
+        </collision>
+        <xacro:inertial_cylinder mass="${scaled_wheel_mass}" radius="${scaled_back_wheel_radius}" length="${scaled_back_wheel_length}">
+            <origin xyz="0 0 ${scaled_back_wheel_length / 2}" rpy="0 0 0"/>
         </xacro:inertial_cylinder>
     </link>
@@ -235,27 +261,25 @@
         <mu2 value="0.001"/>
     </gazebo>
-    <!-- RIGHT FRONT WHEEL LINK -->
     <joint name="rf_wheel_joint" type="fixed">
         <parent link="front_chassis"/>
         <child link="rf_wheel"/>
-        <origin xyz="${scaled_wheel_radius} -${scaled_chassis_radius} 0" rpy="${pi/2} 0 0"/>
-        <!-- <axis xyz="0 0 -1"/> -->
+        <origin xyz="${scaled_back_wheel_radius} -${scaled_back_chassis_radius} 0" rpy="${pi/2} 0 0"/>
     </joint>
     <link name="rf_wheel">
         <visual>
-            <origin xyz="0 0 ${scaled_wheel_length / 2}" rpy="0 0 0"/>
-            <geometry>
-                <cylinder radius="${scaled_wheel_radius}" length="${scaled_wheel_length}"/>
+            <origin xyz="0 0 ${scaled_back_wheel_length / 2}" rpy="0 0 0"/>
+            <geometry>
+                <cylinder radius="${scaled_back_wheel_radius}" length="${scaled_back_wheel_length}"/>
             </geometry>
             <material name="red"/>
         </visual>
         <collision>
-            <origin xyz="0 0 ${scaled_wheel_length / 2}" rpy="0 0 0"/>
-            <geometry>
-                <cylinder radius="${scaled_wheel_radius}" length="${scaled_wheel_length}"/>
-            </geometry>
-        </collision>
-        <xacro:inertial_cylinder mass="${scaled_wheel_mass}" radius="${scaled_wheel_radius}" length="${scaled_wheel_length}">
-            <origin xyz="0 0 ${scaled_wheel_length / 2}" rpy="0 0 0"/>
+            <origin xyz="0 0 ${scaled_back_wheel_length / 2}" rpy="0 0 0"/>
+            <geometry>
+                <cylinder radius="${scaled_back_wheel_radius}" length="${scaled_back_wheel_length}"/>
+            </geometry>
+        </collision>
+        <xacro:inertial_cylinder mass="${scaled_wheel_mass}" radius="${scaled_back_wheel_radius}" length="${scaled_back_wheel_length}">
+            <origin xyz="0 0 ${scaled_back_wheel_length / 2}" rpy="0 0 0"/>
         </xacro:inertial_cylinder>
     </link>
@@ -264,15 +288,14 @@
         <mu1 value="0.001"/>
         <mu2 value="0.001"/>
-    </gazebo>
-    <!-- FRONT CASTER WHEEL LINK -->
+    </gazebo> -->
     <joint name="f_caster_wheel_joint" type="fixed">
         <parent link="front_chassis"/>
         <child link="f_caster_wheel"/>
-        <origin xyz="${scaled_chassis_length * 0.75} 0 -${scaled_wheel_radius / 2}" rpy="0 0 0"/>
+        <origin xyz="${scaled_front_chassis_length * 0.75} 0 -${scaled_front_chassis_radius / 2}" rpy="0 0 0"/>
     </joint>
     <link name="f_caster_wheel">
         <visual>
             <geometry>
-                <sphere radius="${scaled_wheel_radius / 2}"/>
+                <sphere radius="${scaled_front_chassis_radius / 2}"/>
             </geometry>
             <material name="black"/>
@@ -280,8 +303,8 @@
         <collision>
             <geometry>
-                <sphere radius="${scaled_wheel_radius / 2}"/>
-            </geometry>
-        </collision>
-        <xacro:inertial_sphere mass="${scaled_caster_wheel_mass}" radius="${scaled_wheel_radius / 2}">
+                <sphere radius="${scaled_front_chassis_radius / 2}"/>
+            </geometry>
+        </collision>
+        <xacro:inertial_sphere mass="${scaled_caster_wheel_mass}" radius="${scaled_front_chassis_radius / 2}">
             <origin xyz="0 0 0" rpy="0 0 0"/>
         </xacro:inertial_sphere>
@@ -296,5 +319,5 @@
         <parent link="front_chassis"/>
         <child link="camera_link"/>
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
File: description/robot_exe.xacro (robot description, xacro)
@@ -3,5 +3,5 @@
     <xacro:include filename="inertial_macros.xacro"/>
     <xacro:include filename="depth_camera.xacro"/>
-    <xacro:include filename="robot_core_test.xacro"/>
+    <xacro:include filename="robot_core.xacro"/>
     <xacro:include filename="keyboard_control.xacro"/>
     <xacro:include filename="control.xacro"/>
